Commit message: updates to lw

File: kbot-v2-lw-feet/robot.urdf (robot description, URDF)
Before this commit: robot kbotv2p0_nosubassy, 23 links, 22 joints
Joints:
- joint dof_left_hip_roll_03: axis 0 0 -1 -> 0 0 1.0; limit lower=-0.209440 upper=2.268928 effort=60 velocity=6.283 -> lower=-2.268928 upper=0.209440 effort=60 velocity=6.283
- joint dof_left_shoulder_roll_03: axis 0 0 1 -> 0 0 -1.0; limit lower=-0.383972 upper=1.658063 effort=60 velocity=6.283 -> lower=-1.658063 upper=0.383972 effort=60 velocity=6.283
- joint dof_right_hip_roll_03: axis 0 0 -1 -> 0 0 1.0; limit lower=-2.268928 upper=0.209440 effort=60 velocity=6.283 -> lower=-0.209440 upper=2.268928 effort=60 velocity=6.283
- joint dof_right_shoulder_roll_03: axis 0 0 -1 -> 0 0 1.0; limit lower=-1.658063 upper=0.383972 effort=60 velocity=6.283 -> lower=-0.383972 upper=1.658063 effort=60 velocity=6.283

Commit message: no flip for these motors needed

File: kbot-v2-lw-feet/robot.urdf (robot description, URDF)
Before this commit: robot kbotv2p0_nosubassy, 23 links, 22 joints
Joints:
- joint dof_left_hip_roll_03: axis 0 0 1.0 -> 0 0 -1; limit lower=-2.268928 upper=0.209440 effort=60 velocity=6.283 -> lower=-0.209440 upper=2.268928 effort=60 velocity=6.283
- joint dof_left_shoulder_roll_03: axis 0 0 -1.0 -> 0 0 1; limit lower=-1.658063 upper=0.383972 effort=60 velocity=6.283 -> lower=-0.383972 upper=1.658063 effort=60 velocity=6.283
- joint dof_right_hip_roll_03: axis 0 0 1.0 -> 0 0 -1; limit lower=-0.209440 upper=2.268928 effort=60 velocity=6.283 -> lower=-2.268928 upper=0.209440 effort=60 velocity=6.283
- joint dof_right_shoulder_roll_03: axis 0 0 1.0 -> 0 0 -1; limit lower=-0.383972 upper=1.658063 effort=60 velocity=6.283 -> lower=-1.658063 upper=0.383972 effort=60 velocity=6.283

Commit message: fix imu orientation

File: kbot-v2-lw-feet/robot.urdf (robot description, URDF)
Before this commit: robot kbotv2p0_nosubassy, 23 links, 22 joints
Joints:
- joint dof_left_hip_roll_03: axis 0 0 1.0 -> 0 0 -1; limit lower=-2.268928 upper=0.209440 effort=60 velocity=6.283 -> lower=-0.209440 upper=2.268928 effort=60 velocity=6.283
- joint dof_left_shoulder_roll_03: axis 0 0 -1.0 -> 0 0 1; limit lower=-1.658063 upper=0.383972 effort=60 velocity=6.283 -> lower=-0.383972 upper=1.658063 effort=60 velocity=6.283
- joint dof_right_hip_roll_03: axis 0 0 1.0 -> 0 0 -1; limit lower=-0.209440 upper=2.268928 effort=60 velocity=6.283 -> lower=-2.268928 upper=0.209440 effort=60 velocity=6.283
- joint dof_right_shoulder_roll_03: axis 0 0 1.0 -> 0 0 -1; limit lower=-0.383972 upper=1.658063 effort=60 velocity=6.283 -> lower=-1.658063 upper=0.383972 effort=60 velocity=6.283
- joint frame_imu_site: origin xyz=0.123783 0.043292 0.231518 rpy=-1.570796 -0.000002 1.570796 -> xyz=0.121783 0.043292 0.231518 rpy=1.582557 1.570794 1.582557

Commit message: fixkbot direction

File: kbot-v2-lw-feet/robot.urdf (robot description, URDF)
Before this commit: robot kbotv2p0_nosubassy, 23 links, 22 joints
Joints:
- joint floating_base_joint: origin xyz=0 0 0 rpy=0.00 0.00 0.00 -> xyz=0 0 0 rpy=0.00 0.00 1.57

File: kbot-v2-lw/robot.urdf (robot description, URDF)
Before this commit: robot kbotv2p0_nosubassy, 23 links, 22 joints
Joints:
- joint floating_base_joint: origin xyz=0 0 0 rpy=0.00 0.00 0.00 -> xyz=0 0 0 rpy=0.00 0.00 1.57
