Commit message: update zbot 6dof

File: zbot-6dof/robot.urdf (robot description, URDF)
Before this commit: robot top_level_assy_[urdf], 23 links, 22 joints
Links:
- removed link FINGER_1
- removed link FINGER_1_1
- removed link FK_AP_019_25T_11
- removed link FK_AP_019_25T_11_1
- removed link Hip_Bracket
- removed link Hip_Bracket_2
- removed link IMU
- removed link ST15_12
- removed link ST15_13
- removed link ST15_14
- removed link ST15_15
- removed link ST15_4
- removed link ST15_7
- removed link Upper_Leg
- removed link Upper_Leg_2
- removed link Z_BOT2_MASTER_BODY_SKELETON
- removed link Z_BOT2_MASTER_SHOULDER2
- removed link Z_BOT2_MASTER_SHOULDER2_1
- added link IMU_2, mass 0.001887
- added link Left_1910_0025_0816_REV1, mass 0.019227
- added link Left_Ankle_Pitch_ST15, mass 0.217273
- added link Left_Finger, mass 0.022323; collision mesh filename=meshes/Left_Finger.collision.stl; visual mesh filename=meshes/Left_Finger.collision.stl
- added link Left_Hip_Roll_ST15, mass 0.217273; collision mesh filename=meshes/Left_Hip_Roll_ST15.collision.stl; visual mesh filename=meshes/Left_Hip_Roll_ST15.collision.stl
- added link Left_Knee_Pitch_ST15, mass 0.133647; collision mesh filename=meshes/Left_Knee_Pitch_ST15.collision.stl; visual mesh filename=meshes/Left_Knee_Pitch_ST15.collision.stl
- added link Left_Shoulder_Roll_SERVO_DUAL_v5, mass 0.122460; collision mesh filename=meshes/Left_Shoulder_Roll_SERVO_DUAL_v5.collision.stl; visual mesh filename=meshes/Left_Shoulder_Roll_SERVO_DUAL_v5.collision.stl
- added link Left_Upper_Hip_Bracket, mass 0.034227
- added link Left_Upper_Leg, mass 0.030705
- added link Right_1910_0025_0816_REV1, mass 0.019227
- added link Right_Ankle_Pitch_ST15, mass 0.217273
- added link Right_Finger, mass 0.015601; collision mesh filename=meshes/Right_Finger.collision.stl; visual mesh filename=meshes/Right_Finger.collision.stl
- added link Right_Hip_Roll_ST15, mass 0.217273; collision mesh filename=meshes/Right_Hip_Roll_ST15.collision.stl; visual mesh filename=meshes/Right_Hip_Roll_ST15.collision.stl
- added link Right_Knee_Pitch_ST15, mass 0.133647; collision mesh filename=meshes/Right_Knee_Pitch_ST15.collision.stl; visual mesh filename=meshes/Right_Knee_Pitch_ST15.collision.stl
- added link Right_Shoulder_Roll_SERVO_DUAL_v5, mass 0.122460; collision mesh filename=meshes/Right_Shoulder_Roll_SERVO_DUAL_v5.collision.stl; visual mesh filename=meshes/Right_Shoulder_Roll_SERVO_DUAL_v5.collision.stl
- added link Right_Upper_Hip_Bracket, mass 0.022071
- added link Right_Upper_Leg, mass 0.030705
- added link Top_Brace, mass 1.292559; collision mesh filename=meshes/Top_Brace.collision.stl; visual mesh filename=meshes/Top_Brace.collision.stl
- link L_ARM_MIRROR_1: geometry collision mesh filename=meshes/L_ARM_MIRROR_1.collision.stl; visual mesh filename=meshes/L_ARM_MIRROR_1.collision.stl
- link Left_Foot: geometry collision mesh filename=meshes/Left_Foot.collision.stl; visual mesh filename=meshes/Left_Foot.collision.stl
- link R_ARM_MIRROR_1: geometry collision mesh filename=meshes/R_ARM_MIRROR_1.collision.stl; visual mesh filename=meshes/R_ARM_MIRROR_1.collision.stl
- link Right_Foot: geometry collision mesh filename=meshes/Right_Foot.collision.stl; visual mesh filename=meshes/Right_Foot.collision.stl
Joints:
- removed joint imu
- removed joint left_ankle_pitch
- removed joint left_ankle_roll
- removed joint left_elbow_yaw
- removed joint left_gripper
- removed joint left_hip_pitch
- removed joint left_hip_roll
- removed joint left_hip_yaw
- removed joint left_knee_pitch
- removed joint left_shoulder_pitch
- removed joint left_shoulder_yaw
- removed joint right_ankle_pitch
- removed joint right_ankle_roll
- removed joint right_elbow_yaw
- removed joint right_gripper
- removed joint right_hip_pitch
- removed joint right_hip_roll
- removed joint right_hip_yaw
- removed joint right_knee_pitch
- removed joint right_shoulder_pitch
- removed joint right_shoulder_yaw
- added joint IMU: type fixed, parent Top_Brace, child IMU_2, origin xyz=-0.010000 -0.006714 0.034035 rpy=0 0 0
- added joint left_ankle_pitch_50: type revolute, parent Left_Knee_Pitch_ST15, child Left_Ankle_Pitch_ST15, origin xyz=0 0.100000 -0.036040 rpy=-3.141593 0 0, axis 0 0 1, limit lower=-1.396263 upper=0.698132 effort=2 velocity=2
- added joint left_ankle_roll_50: type revolute, parent Left_Ankle_Pitch_ST15, child Left_Foot, origin xyz=0.015150 0 -0.018800 rpy=-3.141593 -1.570796 0, axis 0 0 1, limit lower=-1.047198 upper=1.047198 effort=2 velocity=2
- added joint left_elbow_roll_15: type revolute, parent Left_Shoulder_Roll_SERVO_DUAL_v5, child R_ARM_MIRROR_1, origin xyz=0 0.086212 -0.038650 rpy=0 0 0, axis 0 0 1, limit lower=-0.872665 upper=1.570796 effort=2 velocity=2
- added joint left_gripper_15: type revolute, parent R_ARM_MIRROR_1, child Left_Finger, origin xyz=0.011815 0.066309 0.038340 rpy=-3.141593 0 -0.349066, axis 0 0 1, limit lower=-0.523599 upper=0.523599 effort=2 velocity=2
- added joint left_hip_pitch_50: type revolute, parent Left_Hip_Roll_ST15, child Left_Upper_Leg, origin xyz=-0.019800 0 0.016150 rpy=0 1.570796 0, axis 0 0 1, limit lower=-1.570796 upper=0.872665 effort=2 velocity=2
- added joint left_hip_roll_50: type revolute, parent Left_Upper_Hip_Bracket, child Left_Hip_Roll_ST15, origin xyz=-0.000087 0.019650 -0.026665 rpy=1.570796 0 0, axis 0 0 1, limit lower=-0.610865 upper=0.610865 effort=2 velocity=2
- added joint left_hip_yaw_50: type revolute, parent Top_Brace, child Left_Upper_Hip_Bracket, origin xyz=0.043042 0.000211 -0.089300 rpy=0 0 0, axis 0 0 1, limit lower=-1.570796 upper=1.570796 effort=2 velocity=2
- added joint left_knee_pitch_50: type revolute, parent Left_Upper_Leg, child Left_Knee_Pitch_ST15, origin xyz=0 -0.100000 0.001260 rpy=3.141593 0 0, axis 0 0 1, limit lower=-1.396263 upper=1.396263 effort=2 velocity=2
- added joint left_shoulder_pitch_15: type revolute, parent Top_Brace, child Left_1910_0025_0816_REV1, origin xyz=0.060300 0.000211 0.026100 rpy=-1.570796 0 1.570796, axis 0 0 1, limit lower=-1.570796 upper=3.141593 effort=2 velocity=2
- added joint left_shoulder_roll_15: type revolute, parent Left_1910_0025_0816_REV1, child Left_Shoulder_Roll_SERVO_DUAL_v5, origin xyz=0.017892 0.004100 -0.032700 rpy=0 1.570796 0, axis 0 0 1, limit lower=-2.617994 upper=0.401426 effort=2 velocity=2
- added joint right_ankle_pitch_50: type revolute, parent Right_Knee_Pitch_ST15, child Right_Ankle_Pitch_ST15, origin xyz=0 0.100000 -0.036859 rpy=-3.141593 0 0, axis 0 0 1, limit lower=-1.396263 upper=0.698132 effort=2 velocity=2
- added joint right_ankle_roll_50: type revolute, parent Right_Ankle_Pitch_ST15, child Right_Foot, origin xyz=0.015150 0 -0.018800 rpy=-3.141593 -1.570796 0, axis 0 0 1, limit lower=-1.047198 upper=1.047198 effort=2 velocity=2
- added joint right_elbow_roll_15: type revolute, parent Right_Shoulder_Roll_SERVO_DUAL_v5, child L_ARM_MIRROR_1, origin xyz=0 -0.086212 0.001000 rpy=0 0 0, axis 0 0 -1, limit lower=-0.872665 upper=1.570796 effort=2 velocity=2
- added joint right_gripper_15: type revolute, parent L_ARM_MIRROR_1, child Right_Finger, origin xyz=-0.011778 -0.066206 0.001260 rpy=-3.141593 0 -0.349066, axis 0 0 1, limit lower=-0.523599 upper=0.523599 effort=2 velocity=2
- added joint right_hip_pitch_50: type revolute, parent Right_Hip_Roll_ST15, child Right_Upper_Leg, origin xyz=-0.019800 0 0.016150 rpy=0 1.570796 0, axis 0 0 1, limit lower=-1.570796 upper=0.872665 effort=2 velocity=2
- added joint right_hip_roll_50: type revolute, parent Right_Upper_Hip_Bracket, child Right_Hip_Roll_ST15, origin xyz=-0.000087 0.019650 -0.026665 rpy=1.570796 0 0, axis 0 0 1, limit lower=-0.610865 upper=0.610865 effort=2 velocity=2
- added joint right_hip_yaw_50: type revolute, parent Top_Brace, child Right_Upper_Hip_Bracket, origin xyz=-0.043042 0.000211 -0.089300 rpy=0 0 0, axis 0 0 1, limit lower=-1.570796 upper=1.570796 effort=2 velocity=2
- added joint right_knee_pitch_50: type revolute, parent Right_Upper_Leg, child Right_Knee_Pitch_ST15, origin xyz=0 -0.100000 0.001260 rpy=3.141593 0 0, axis 0 0 1, limit lower=-1.396263 upper=1.396263 effort=2 velocity=2
- added joint right_shoulder_pitch_15: type revolute, parent Top_Brace, child Right_1910_0025_0816_REV1, origin xyz=-0.060300 0.000211 0.026100 rpy=1.570796 0 1.570796, axis 0 0 1, limit lower=-1.570796 upper=3.141593 effort=2 velocity=2
- added joint right_shoulder_roll_15: type revolute, parent Right_1910_0025_0816_REV1, child Right_Shoulder_Roll_SERVO_DUAL_v5, origin xyz=-0.017758 -0.004100 -0.032700 rpy=0 -1.570796 0, axis 0 0 1, limit lower=-2.617994 upper=0.401426 effort=2 velocity=2
- joint floating_base_joint: child Z_BOT2_MASTER_BODY_SKELETON -> Top_Brace

Commit message: update zbot 6dof urdf

File: zbot-6dof/robot.urdf (robot description, URDF)
Before this commit: robot v3.1_top_level_assembly_[urdf], 23 links, 22 joints
Links:
- removed link IMU_2
- added link imu, mass 0.001887; visual mesh filename=meshes/imu.stl
- link L_ARM_MIRROR_1: geometry collision mesh filename=meshes/L_ARM_MIRROR_1.collision.stl; visual mesh filename=meshes/L_ARM_MIRROR_1.stl
- link Left_1910_0025_0816_REV1: geometry visual mesh filename=meshes/Left_1910_0025_0816_REV1.stl
- link Left_Ankle_Pitch_ST15: geometry visual mesh filename=meshes/Left_Ankle_Pitch_ST15.stl
- link Left_Finger: geometry collision mesh filename=meshes/Left_Finger.collision.stl; visual mesh filename=meshes/Left_Finger.stl
- link Left_Foot: geometry collision mesh filename=meshes/Left_Foot.collision.stl; visual mesh filename=meshes/Left_Foot.stl
- link Left_Hip_Roll_ST15: geometry collision mesh filename=meshes/Left_Hip_Roll_ST15.collision.stl; visual mesh filename=meshes/Left_Hip_Roll_ST15.stl
- link Left_Knee_Pitch_ST15: geometry collision mesh filename=meshes/Left_Knee_Pitch_ST15.collision.stl; visual mesh filename=meshes/Left_Knee_Pitch_ST15.stl
- link Left_Shoulder_Roll_SERVO_DUAL_v5: geometry collision mesh filename=meshes/Left_Shoulder_Roll_SERVO_DUAL_v5.collision.stl; visual mesh filename=meshes/Left_Shoulder_Roll_SERVO_DUAL_v5.stl
- link Left_Upper_Hip_Bracket: geometry visual mesh filename=meshes/Left_Upper_Hip_Bracket.stl
- link Left_Upper_Leg: geometry visual mesh filename=meshes/Left_Upper_Leg.stl
- link R_ARM_MIRROR_1: geometry collision mesh filename=meshes/R_ARM_MIRROR_1.collision.stl; visual mesh filename=meshes/R_ARM_MIRROR_1.stl
- link Right_1910_0025_0816_REV1: geometry visual mesh filename=meshes/Right_1910_0025_0816_REV1.stl
- link Right_Ankle_Pitch_ST15: geometry visual mesh filename=meshes/Right_Ankle_Pitch_ST15.stl
- link Right_Finger: geometry collision mesh filename=meshes/Right_Finger.collision.stl; visual mesh filename=meshes/Right_Finger.stl
- link Right_Foot: geometry collision mesh filename=meshes/Right_Foot.collision.stl; visual mesh filename=meshes/Right_Foot.stl
- link Right_Hip_Roll_ST15: geometry collision mesh filename=meshes/Right_Hip_Roll_ST15.collision.stl; visual mesh filename=meshes/Right_Hip_Roll_ST15.stl
- link Right_Knee_Pitch_ST15: geometry collision mesh filename=meshes/Right_Knee_Pitch_ST15.collision.stl; visual mesh filename=meshes/Right_Knee_Pitch_ST15.stl
- link Right_Shoulder_Roll_SERVO_DUAL_v5: geometry collision mesh filename=meshes/Right_Shoulder_Roll_SERVO_DUAL_v5.collision.stl; visual mesh filename=meshes/Right_Shoulder_Roll_SERVO_DUAL_v5.stl
- link Right_Upper_Hip_Bracket: geometry visual mesh filename=meshes/Right_Upper_Hip_Bracket.stl
- link Right_Upper_Leg: geometry visual mesh filename=meshes/Right_Upper_Leg.stl
- link Top_Brace: geometry collision mesh filename=meshes/Top_Brace.collision.stl; visual mesh filename=meshes/Top_Brace.stl
Joints:
- removed joint IMU
- added joint frame_imu_site: type fixed, parent Top_Brace, child imu, origin xyz=-0.010000 0.008286 0.034035 rpy=0 0 -1.570796

Commit message: zbot 6dof

File: zbot-6dof/robot.urdf (robot description, URDF)
Before this commit: robot v3.1_top_level_assembly_[urdf], 23 links, 22 joints
Links:
- removed link Left_Ankle_Pitch_ST15
- removed link Left_Hip_Roll_ST15
- removed link Left_Knee_Pitch_ST15
- removed link Left_Shoulder_Roll_SERVO_DUAL_v5
- removed link Right_Ankle_Pitch_ST15
- removed link Right_Hip_Roll_ST15
- removed link Right_Knee_Pitch_ST15
- removed link Right_Shoulder_Roll_SERVO_DUAL_v5
- added link Left_Ankle_Pitch_STS3250, mass 0.178551; visual mesh filename=meshes/Left_Ankle_Pitch_STS3250.stl
- added link Left_Hip_Roll_STS3250, mass 0.178551; collision mesh filename=meshes/Left_Hip_Roll_STS3250.collision.stl; visual mesh filename=meshes/Left_Hip_Roll_STS3250.stl
- added link Left_Knee_Pitch_STS3250, mass 0.114286; collision mesh filename=meshes/Left_Knee_Pitch_STS3250.collision.stl; visual mesh filename=meshes/Left_Knee_Pitch_STS3250.stl
- added link Left_Shoulder_Roll_STS3250, mass 0.142460; collision mesh filename=meshes/Left_Shoulder_Roll_STS3250.collision.stl; visual mesh filename=meshes/Left_Shoulder_Roll_STS3250.stl
- added link Right_Ankle_Pitch_STS3250, mass 0.178551; visual mesh filename=meshes/Right_Ankle_Pitch_STS3250.stl
- added link Right_Hip_Roll_STS3250, mass 0.178551; collision mesh filename=meshes/Right_Hip_Roll_STS3250.collision.stl; visual mesh filename=meshes/Right_Hip_Roll_STS3250.stl
- added link Right_Knee_Pitch_STS3250, mass 0.114286; collision mesh filename=meshes/Right_Knee_Pitch_STS3250.collision.stl; visual mesh filename=meshes/Right_Knee_Pitch_STS3250.stl
- added link Right_Shoulder_Roll_STS3250, mass 0.142460; collision mesh filename=meshes/Right_Shoulder_Roll_STS3250.collision.stl; visual mesh filename=meshes/Right_Shoulder_Roll_STS3250.stl
- link L_ARM_MIRROR_1: mass 0.153130 -> 0.184048
- link Left_Finger: mass 0.022323 -> 0.044365
- link R_ARM_MIRROR_1: mass 0.153130 -> 0.184048
- link Right_Finger: mass 0.015601 -> 0.044365
- link Top_Brace: mass 1.292559 -> 1.309559
Joints:
- joint frame_imu_site: origin xyz=-0.010000 0.008286 0.036035 rpy=-3.141593 0 -1.570796 -> xyz=-0.010000 0.008286 0.036035 rpy=-3.141593 0 3.141593
- joint left_ankle_pitch: child Left_Ankle_Pitch_ST15 -> Left_Ankle_Pitch_STS3250; parent Left_Knee_Pitch_ST15 -> Left_Knee_Pitch_STS3250
- joint left_ankle_roll: parent Left_Ankle_Pitch_ST15 -> Left_Ankle_Pitch_STS3250
- joint left_elbow_roll: parent Left_Shoulder_Roll_SERVO_DUAL_v5 -> Left_Shoulder_Roll_STS3250
- joint left_hip_pitch: parent Left_Hip_Roll_ST15 -> Left_Hip_Roll_STS3250
- joint left_hip_roll: child Left_Hip_Roll_ST15 -> Left_Hip_Roll_STS3250
- joint left_knee_pitch: child Left_Knee_Pitch_ST15 -> Left_Knee_Pitch_STS3250
- joint left_shoulder_roll: child Left_Shoulder_Roll_SERVO_DUAL_v5 -> Left_Shoulder_Roll_STS3250
- joint right_ankle_pitch: child Right_Ankle_Pitch_ST15 -> Right_Ankle_Pitch_STS3250; parent Right_Knee_Pitch_ST15 -> Right_Knee_Pitch_STS3250
- joint right_ankle_roll: parent Right_Ankle_Pitch_ST15 -> Right_Ankle_Pitch_STS3250
- joint right_elbow_roll: parent Right_Shoulder_Roll_SERVO_DUAL_v5 -> Right_Shoulder_Roll_STS3250
- joint right_hip_pitch: parent Right_Hip_Roll_ST15 -> Right_Hip_Roll_STS3250
- joint right_hip_roll: child Right_Hip_Roll_ST15 -> Right_Hip_Roll_STS3250
- joint right_knee_pitch: child Right_Knee_Pitch_ST15 -> Right_Knee_Pitch_STS3250
- joint right_shoulder_roll: child Right_Shoulder_Roll_SERVO_DUAL_v5 -> Right_Shoulder_Roll_STS3250
