Commit message: zbot imu and joshuas changes

File: zbot-6dof-feet/robot.urdf (robot description, URDF)
Before this commit: robot v3.1_top_level_assembly_[urdf], 23 links, 22 joints
Links:
- removed link Left_Ankle_Pitch_ST15
- removed link Left_Hip_Roll_ST15
- removed link Left_Knee_Pitch_ST15
- removed link Left_Shoulder_Roll_SERVO_DUAL_v5
- removed link Right_Ankle_Pitch_ST15
- removed link Right_Hip_Roll_ST15
- removed link Right_Knee_Pitch_ST15
- removed link Right_Shoulder_Roll_SERVO_DUAL_v5
- added link Left_Ankle_Pitch_STS3250, mass 0.178551; visual mesh filename=meshes/Left_Ankle_Pitch_STS3250.stl
- added link Left_Hip_Roll_STS3250, mass 0.178551; visual mesh filename=meshes/Left_Hip_Roll_STS3250.stl
- added link Left_Knee_Pitch_STS3250, mass 0.114286; visual mesh filename=meshes/Left_Knee_Pitch_STS3250.stl
- added link Left_Shoulder_Roll_STS3250, mass 0.142460; visual mesh filename=meshes/Left_Shoulder_Roll_STS3250.stl
- added link Right_Ankle_Pitch_STS3250, mass 0.178551; visual mesh filename=meshes/Right_Ankle_Pitch_STS3250.stl
- added link Right_Hip_Roll_STS3250, mass 0.178551; visual mesh filename=meshes/Right_Hip_Roll_STS3250.stl
- added link Right_Knee_Pitch_STS3250, mass 0.114286; visual mesh filename=meshes/Right_Knee_Pitch_STS3250.stl
- added link Right_Shoulder_Roll_STS3250, mass 0.142460; visual mesh filename=meshes/Right_Shoulder_Roll_STS3250.stl
- link L_ARM_MIRROR_1: mass 0.153130 -> 0.184048
- link Left_Finger: mass 0.022323 -> 0.044365
- link R_ARM_MIRROR_1: mass 0.153130 -> 0.184048
- link Right_Finger: mass 0.015601 -> 0.044365
- link Top_Brace: mass 1.292559 -> 1.309559
Joints:
- joint frame_imu_site: origin xyz=-0.010000 0.008286 0.036035 rpy=-3.141593 0 -1.570796 -> xyz=-0.010000 0.008286 0.036035 rpy=-3.141593 0 3.141593
- joint left_ankle_pitch: child Left_Ankle_Pitch_ST15 -> Left_Ankle_Pitch_STS3250; parent Left_Knee_Pitch_ST15 -> Left_Knee_Pitch_STS3250
- joint left_ankle_roll: parent Left_Ankle_Pitch_ST15 -> Left_Ankle_Pitch_STS3250
- joint left_elbow_roll: parent Left_Shoulder_Roll_SERVO_DUAL_v5 -> Left_Shoulder_Roll_STS3250
- joint left_hip_pitch: parent Left_Hip_Roll_ST15 -> Left_Hip_Roll_STS3250
- joint left_hip_roll: child Left_Hip_Roll_ST15 -> Left_Hip_Roll_STS3250
- joint left_knee_pitch: child Left_Knee_Pitch_ST15 -> Left_Knee_Pitch_STS3250
- joint left_shoulder_roll: child Left_Shoulder_Roll_SERVO_DUAL_v5 -> Left_Shoulder_Roll_STS3250
- joint right_ankle_pitch: child Right_Ankle_Pitch_ST15 -> Right_Ankle_Pitch_STS3250; parent Right_Knee_Pitch_ST15 -> Right_Knee_Pitch_STS3250
- joint right_ankle_roll: parent Right_Ankle_Pitch_ST15 -> Right_Ankle_Pitch_STS3250
- joint right_elbow_roll: parent Right_Shoulder_Roll_SERVO_DUAL_v5 -> Right_Shoulder_Roll_STS3250
- joint right_hip_pitch: parent Right_Hip_Roll_ST15 -> Right_Hip_Roll_STS3250
- joint right_hip_roll: child Right_Hip_Roll_ST15 -> Right_Hip_Roll_STS3250
- joint right_knee_pitch: child Right_Knee_Pitch_ST15 -> Right_Knee_Pitch_STS3250
- joint right_shoulder_roll: child Right_Shoulder_Roll_SERVO_DUAL_v5 -> Right_Shoulder_Roll_STS3250

Commit message: new imu corection

File: zbot-6dof-feet/robot.urdf (robot description, URDF)
Before this commit: robot [urdf]_v3.1_top_level_assembly, 23 links, 22 joints
Joints:
- joint frame_imu_site: origin xyz=-0.010000 0.008286 0.036035 rpy=-3.141593 0 3.141593 -> xyz=-0.010000 0.008286 0.036035 rpy=-3.141593 0 0

File: zbot-6dof/robot.urdf (robot description, URDF)
Before this commit: robot [urdf]_v3.1_top_level_assembly, 23 links, 22 joints
Joints:
- joint frame_imu_site: origin xyz=-0.010000 0.008286 0.036035 rpy=-3.141593 0 3.141593 -> xyz=-0.010000 0.008286 0.036035 rpy=-3.141593 0 0

Commit message: zbot imu pose correction and joshuas changes (#27)
* zbot imu and joshuas changes

* zbot 6dof

* new imu corection

File: zbot-6dof-feet/robot.urdf (robot description, URDF)
Before this commit: robot v3.1_top_level_assembly_[urdf], 23 links, 22 joints
Links:
- removed link Left_Ankle_Pitch_ST15
- removed link Left_Hip_Roll_ST15
- removed link Left_Knee_Pitch_ST15
- removed link Left_Shoulder_Roll_SERVO_DUAL_v5
- removed link Right_Ankle_Pitch_ST15
- removed link Right_Hip_Roll_ST15
- removed link Right_Knee_Pitch_ST15
- removed link Right_Shoulder_Roll_SERVO_DUAL_v5
- added link Left_Ankle_Pitch_STS3250, mass 0.178551; visual mesh filename=meshes/Left_Ankle_Pitch_STS3250.stl
- added link Left_Hip_Roll_STS3250, mass 0.178551; visual mesh filename=meshes/Left_Hip_Roll_STS3250.stl
- added link Left_Knee_Pitch_STS3250, mass 0.114286; visual mesh filename=meshes/Left_Knee_Pitch_STS3250.stl
- added link Left_Shoulder_Roll_STS3250, mass 0.142460; visual mesh filename=meshes/Left_Shoulder_Roll_STS3250.stl
- added link Right_Ankle_Pitch_STS3250, mass 0.178551; visual mesh filename=meshes/Right_Ankle_Pitch_STS3250.stl
- added link Right_Hip_Roll_STS3250, mass 0.178551; visual mesh filename=meshes/Right_Hip_Roll_STS3250.stl
- added link Right_Knee_Pitch_STS3250, mass 0.114286; visual mesh filename=meshes/Right_Knee_Pitch_STS3250.stl
- added link Right_Shoulder_Roll_STS3250, mass 0.142460; visual mesh filename=meshes/Right_Shoulder_Roll_STS3250.stl
- link L_ARM_MIRROR_1: mass 0.153130 -> 0.184048
- link Left_Finger: mass 0.022323 -> 0.044365
- link R_ARM_MIRROR_1: mass 0.153130 -> 0.184048
- link Right_Finger: mass 0.015601 -> 0.044365
- link Top_Brace: mass 1.292559 -> 1.309559
Joints:
- joint frame_imu_site: origin xyz=-0.010000 0.008286 0.036035 rpy=-3.141593 0 -1.570796 -> xyz=-0.010000 0.008286 0.036035 rpy=-3.141593 0 0
- joint left_ankle_pitch: child Left_Ankle_Pitch_ST15 -> Left_Ankle_Pitch_STS3250; parent Left_Knee_Pitch_ST15 -> Left_Knee_Pitch_STS3250
- joint left_ankle_roll: parent Left_Ankle_Pitch_ST15 -> Left_Ankle_Pitch_STS3250
- joint left_elbow_roll: parent Left_Shoulder_Roll_SERVO_DUAL_v5 -> Left_Shoulder_Roll_STS3250
- joint left_hip_pitch: parent Left_Hip_Roll_ST15 -> Left_Hip_Roll_STS3250
- joint left_hip_roll: child Left_Hip_Roll_ST15 -> Left_Hip_Roll_STS3250
- joint left_knee_pitch: child Left_Knee_Pitch_ST15 -> Left_Knee_Pitch_STS3250
- joint left_shoulder_roll: child Left_Shoulder_Roll_SERVO_DUAL_v5 -> Left_Shoulder_Roll_STS3250
- joint right_ankle_pitch: child Right_Ankle_Pitch_ST15 -> Right_Ankle_Pitch_STS3250; parent Right_Knee_Pitch_ST15 -> Right_Knee_Pitch_STS3250
- joint right_ankle_roll: parent Right_Ankle_Pitch_ST15 -> Right_Ankle_Pitch_STS3250
- joint right_elbow_roll: parent Right_Shoulder_Roll_SERVO_DUAL_v5 -> Right_Shoulder_Roll_STS3250
- joint right_hip_pitch: parent Right_Hip_Roll_ST15 -> Right_Hip_Roll_STS3250
- joint right_hip_roll: child Right_Hip_Roll_ST15 -> Right_Hip_Roll_STS3250
- joint right_knee_pitch: child Right_Knee_Pitch_ST15 -> Right_Knee_Pitch_STS3250
- joint right_shoulder_roll: child Right_Shoulder_Roll_SERVO_DUAL_v5 -> Right_Shoulder_Roll_STS3250

File: zbot-6dof/robot.urdf (robot description, URDF)
Before this commit: robot v3.1_top_level_assembly_[urdf], 23 links, 22 joints
Links:
- removed link Left_Ankle_Pitch_ST15
- removed link Left_Hip_Roll_ST15
- removed link Left_Knee_Pitch_ST15
- removed link Left_Shoulder_Roll_SERVO_DUAL_v5
- removed link Right_Ankle_Pitch_ST15
- removed link Right_Hip_Roll_ST15
- removed link Right_Knee_Pitch_ST15
- removed link Right_Shoulder_Roll_SERVO_DUAL_v5
- added link Left_Ankle_Pitch_STS3250, mass 0.178551; visual mesh filename=meshes/Left_Ankle_Pitch_STS3250.stl
- added link Left_Hip_Roll_STS3250, mass 0.178551; collision mesh filename=meshes/Left_Hip_Roll_STS3250.collision.stl; visual mesh filename=meshes/Left_Hip_Roll_STS3250.stl
- added link Left_Knee_Pitch_STS3250, mass 0.114286; collision mesh filename=meshes/Left_Knee_Pitch_STS3250.collision.stl; visual mesh filename=meshes/Left_Knee_Pitch_STS3250.stl
- added link Left_Shoulder_Roll_STS3250, mass 0.142460; collision mesh filename=meshes/Left_Shoulder_Roll_STS3250.collision.stl; visual mesh filename=meshes/Left_Shoulder_Roll_STS3250.stl
- added link Right_Ankle_Pitch_STS3250, mass 0.178551; visual mesh filename=meshes/Right_Ankle_Pitch_STS3250.stl
- added link Right_Hip_Roll_STS3250, mass 0.178551; collision mesh filename=meshes/Right_Hip_Roll_STS3250.collision.stl; visual mesh filename=meshes/Right_Hip_Roll_STS3250.stl
- added link Right_Knee_Pitch_STS3250, mass 0.114286; collision mesh filename=meshes/Right_Knee_Pitch_STS3250.collision.stl; visual mesh filename=meshes/Right_Knee_Pitch_STS3250.stl
- added link Right_Shoulder_Roll_STS3250, mass 0.142460; collision mesh filename=meshes/Right_Shoulder_Roll_STS3250.collision.stl; visual mesh filename=meshes/Right_Shoulder_Roll_STS3250.stl
- link L_ARM_MIRROR_1: mass 0.153130 -> 0.184048
- link Left_Finger: mass 0.022323 -> 0.044365
- link R_ARM_MIRROR_1: mass 0.153130 -> 0.184048
- link Right_Finger: mass 0.015601 -> 0.044365
- link Top_Brace: mass 1.292559 -> 1.309559
Joints:
- joint frame_imu_site: origin xyz=-0.010000 0.008286 0.036035 rpy=-3.141593 0 -1.570796 -> xyz=-0.010000 0.008286 0.036035 rpy=-3.141593 0 0
- joint left_ankle_pitch: child Left_Ankle_Pitch_ST15 -> Left_Ankle_Pitch_STS3250; parent Left_Knee_Pitch_ST15 -> Left_Knee_Pitch_STS3250
- joint left_ankle_roll: parent Left_Ankle_Pitch_ST15 -> Left_Ankle_Pitch_STS3250
- joint left_elbow_roll: parent Left_Shoulder_Roll_SERVO_DUAL_v5 -> Left_Shoulder_Roll_STS3250
- joint left_hip_pitch: parent Left_Hip_Roll_ST15 -> Left_Hip_Roll_STS3250
- joint left_hip_roll: child Left_Hip_Roll_ST15 -> Left_Hip_Roll_STS3250
- joint left_knee_pitch: child Left_Knee_Pitch_ST15 -> Left_Knee_Pitch_STS3250
- joint left_shoulder_roll: child Left_Shoulder_Roll_SERVO_DUAL_v5 -> Left_Shoulder_Roll_STS3250
- joint right_ankle_pitch: child Right_Ankle_Pitch_ST15 -> Right_Ankle_Pitch_STS3250; parent Right_Knee_Pitch_ST15 -> Right_Knee_Pitch_STS3250
- joint right_ankle_roll: parent Right_Ankle_Pitch_ST15 -> Right_Ankle_Pitch_STS3250
- joint right_elbow_roll: parent Right_Shoulder_Roll_SERVO_DUAL_v5 -> Right_Shoulder_Roll_STS3250
- joint right_hip_pitch: parent Right_Hip_Roll_ST15 -> Right_Hip_Roll_STS3250
- joint right_hip_roll: child Right_Hip_Roll_ST15 -> Right_Hip_Roll_STS3250
- joint right_knee_pitch: child Right_Knee_Pitch_ST15 -> Right_Knee_Pitch_STS3250
- joint right_shoulder_roll: child Right_Shoulder_Roll_SERVO_DUAL_v5 -> Right_Shoulder_Roll_STS3250

Commit message: zbot updates new flips

File: zbot-6dof-feet/robot.urdf (robot description, URDF)
Before this commit: robot [urdf]_v3.1_top_level_assembly, 23 links, 22 joints
Joints:
- joint right_ankle_pitch: axis 0 0 -1.0 -> 0 0 1; limit lower=-0.698132 upper=1.396263 effort=2 velocity=2 -> lower=-1.396263 upper=0.698132 effort=2 velocity=2
- joint right_hip_yaw: axis 0 0 -1.0 -> 0 0 1

File: zbot-6dof/robot.urdf (robot description, URDF)
Before this commit: robot [urdf]_v3.1_top_level_assembly, 23 links, 22 joints
Joints:
- joint right_ankle_pitch: axis 0 0 -1.0 -> 0 0 1; limit lower=-0.698132 upper=1.396263 effort=2 velocity=2 -> lower=-1.396263 upper=0.698132 effort=2 velocity=2
- joint right_hip_yaw: axis 0 0 -1.0 -> 0 0 1
