Commit message: add back kbot-v1-feet files

File: kbot-v1-feet/robot.urdf (robot description, URDF)
Before this commit: robot k-bot_sim, 71 links, 70 joints
Links:
- removed link link:Hand_(1):hand_actuator_(1)
- removed link link:Hand_(1):hand_part2_(1)
- removed link link:Hand_(1):hand_part_(1)
- removed link link:Hand_(1):hand_shell2_(1)
- removed link link:Hand_(1):hand_shell_(1)
- removed link link:Hand_(1):hand_umi2_(1)
- removed link link:Hand_(1):hand_umi_(1)
- removed link link:Hand_(2):hand_actuator_(1)
- removed link link:Hand_(2):hand_part2_(1)
- removed link link:Hand_(2):hand_part_(1)
- removed link link:Hand_(2):hand_shell2_(1)
- removed link link:Hand_(2):hand_shell_(1)
- removed link link:Hand_(2):hand_umi2_(1)
- removed link link:Hand_(2):hand_umi_(1)
- removed link link:Torso_Naked_(1):body1-part_(1)
- removed link link:Torso_Naked_(1):body1-part_(10)
- removed link link:Torso_Naked_(1):body1-part_(11)
- removed link link:Torso_Naked_(1):body1-part_(12)
- removed link link:Torso_Naked_(1):body1-part_(13)
- removed link link:Torso_Naked_(1):body1-part_(14)
- removed link link:Torso_Naked_(1):body1-part_(2)
- removed link link:Torso_Naked_(1):body1-part_(3)
- removed link link:Torso_Naked_(1):body1-part_(4)
- removed link link:Torso_Naked_(1):body1-part_(5)
- removed link link:Torso_Naked_(1):body1-part_(6)
- removed link link:Torso_Naked_(1):body1-part_(7)
- removed link link:Torso_Naked_(1):body1-part_(8)
- removed link link:Torso_Naked_(1):body1-part_(9)
- removed link link:arm0_(1):shoulder_(3)
- removed link link:arm0_(1):shoulder_(4)
- removed link link:arm0_(1):shoulder_(5)
- removed link link:arm0_(1):shoulder_(6)
- removed link link:arm1_(1):arm-actuator_(1)
- removed link link:arm1_(1):arm-actuator_(2)
- removed link link:arm1_(1):arm1_top_(1)
- removed link link:arm1_(1):arm1_top_2_(2)
- removed link link:arm2_(1):arm2_actuator_(1)
- removed link link:arm2_(1):arm2_shell_(1)
- removed link link:arm2_(2):arm2_actuator_(1)
- removed link link:arm2_(2):arm2_shell_(1)
- removed link link:arm3_(1):arm3_actuator2_(2)
- removed link link:arm3_(1):arm3_actuator_(1)
- removed link link:arm3_(1):arm3_shell2_(1)
- removed link link:arm3_(1):arm3_shell_(1)
- removed link link:foot_flat_(1):foot1_(1)
- removed link link:foot_flat_(1):foot2_(1)
- removed link link:foot_flat_(1):foot3_(2)
- removed link link:foot_flat_(1):foot4_(1)
- removed link link:imu_(1)
- removed link link:leg0_(1):leg0_actuator_(1)
- removed link link:leg0_(1):leg0_bearing_(1)
- removed link link:leg0_(1):leg0_shell_(1)
- removed link link:leg0_(2):leg0_actuator_(1)
- removed link link:leg0_(2):leg0_bearing_(1)
- removed link link:leg0_(2):leg0_shell_(1)
- removed link link:leg1_(1):leg1_actuator2_(2)
- removed link link:leg1_(1):leg1_actuator_(1)
- removed link link:leg1_(1):leg1_shell3_(2)
- removed link link:leg1_(1):leg1_shell_(1)
- removed link link:leg2_(1):leg2_actuator_(1)
- removed link link:leg2_(1):leg2_bearing_(1)
- removed link link:leg2_(1):leg2_shell_(1)
- removed link link:leg2_(2):leg2_actuator_(1)
- removed link link:leg2_(2):leg2_bearing_(1)
- removed link link:leg2_(2):leg2_shell_(1)
- removed link link:leg3_(1):leg3_actuator2_(2)
- removed link link:leg3_(1):leg3_actuator_(1)
- removed link link:leg3_(1):leg3_shell11_(2)
- removed link link:leg3_(1):leg3_shell1_(1)
- removed link link:leg3_(1):leg3_shell33_(2)
- removed link link:leg3_(1):leg3_shell3_(1)
- added link arm1_top, mass 0.572732; visual mesh filename=meshes/arm1_top.stl
- added link arm1_top_2, mass 0.572732; visual mesh filename=meshes/arm1_top_2.stl
- added link arm2_shell, mass 0.510678; visual mesh filename=meshes/arm2_shell.stl
- added link arm2_shell_2, mass 0.510678; visual mesh filename=meshes/arm2_shell_2.stl
- added link arm3_shell, mass 0.578536; visual mesh filename=meshes/arm3_shell.stl
- added link arm3_shell2, mass 0.578536; visual mesh filename=meshes/arm3_shell2.stl
- added link body1_part, mass 9.415838; visual mesh filename=meshes/body1_part.stl
- added link floating_base_link, mass 0.001; visual sphere radius=0.01
- added link foot1, mass 0.582091; collision mesh filename=meshes/foot1.collision.stl; visual mesh filename=meshes/foot1.stl
- added link foot3, mass 0.582091; collision mesh filename=meshes/foot3.collision.stl; visual mesh filename=meshes/foot3.stl
- added link hand_shell, mass 0.793063; visual mesh filename=meshes/hand_shell.stl
- added link hand_shell_2, mass 0.793063; visual mesh filename=meshes/hand_shell_2.stl
- added link imu, mass 0.010000; visual mesh filename=meshes/imu.stl
- added link leg0_shell, mass 1.323448; visual mesh filename=meshes/leg0_shell.stl
- added link leg0_shell_2, mass 1.323448; visual mesh filename=meshes/leg0_shell_2.stl
- added link leg1_shell, mass 1.264352; visual mesh filename=meshes/leg1_shell.stl
- added link leg1_shell3, mass 1.264352; visual mesh filename=meshes/leg1_shell3.stl
- added link leg2_shell, mass 1.820923; visual mesh filename=meshes/leg2_shell.stl
- added link leg2_shell_2, mass 1.820923; visual mesh filename=meshes/leg2_shell_2.stl
- added link leg3_shell1, mass 1.109955; visual mesh filename=meshes/leg3_shell1.stl
- added link leg3_shell11, mass 1.109962; visual mesh filename=meshes/leg3_shell11.stl
- added link shoulder, mass 1.107356; visual mesh filename=meshes/shoulder.stl
- added link shoulder_2, mass 1.107354; visual mesh filename=meshes/shoulder_2.stl
Joints:
- removed joint joint:Hand_(1):Fastened_1
- removed joint joint:Hand_(1):Fastened_2
- removed joint joint:Hand_(1):Fastened_3
- removed joint joint:Hand_(1):Fastened_4
- removed joint joint:Hand_(1):Fastened_5
- removed joint joint:Hand_(1):Fastened_6
- removed joint joint:Hand_(2):Fastened_1
- removed joint joint:Hand_(2):Fastened_2
- removed joint joint:Hand_(2):Fastened_3
- removed joint joint:Hand_(2):Fastened_4
- removed joint joint:Hand_(2):Fastened_5
- removed joint joint:Hand_(2):Fastened_6
- removed joint joint:Torso_Naked_(1):Fastened_1
- removed joint joint:Torso_Naked_(1):Fastened_10
- removed joint joint:Torso_Naked_(1):Fastened_11
- removed joint joint:Torso_Naked_(1):Fastened_16
- removed joint joint:Torso_Naked_(1):Fastened_17
- removed joint joint:Torso_Naked_(1):Fastened_2
- removed joint joint:Torso_Naked_(1):Fastened_3
- removed joint joint:Torso_Naked_(1):Fastened_4
- removed joint joint:Torso_Naked_(1):Fastened_5
- removed joint joint:Torso_Naked_(1):Fastened_6
- removed joint joint:Torso_Naked_(1):Fastened_7
- removed joint joint:Torso_Naked_(1):Fastened_8
- removed joint joint:Torso_Naked_(1):Fastened_9
- removed joint joint:arm0_(1):Fastened_1
- removed joint joint:arm0_(1):Fastened_2
- removed joint joint:arm1_(1):Fastened_1
- removed joint joint:arm1_(1):Fastened_2
- removed joint joint:arm2_(1):Fastened_1
- removed joint joint:arm2_(2):Fastened_1
- removed joint joint:arm3_(1):Fastened_1
- removed joint joint:arm3_(1):Fastened_2
- removed joint joint:foot_flat_(1):Fastened_1
- removed joint joint:foot_flat_(1):Fastened_2
- removed joint joint:imu_link
- removed joint joint:left_ankle_02
- removed joint joint:left_elbow_02
- removed joint joint:left_hip_pitch_04
- removed joint joint:left_hip_roll_03
- removed joint joint:left_hip_yaw_03
- removed joint joint:left_knee_04
- removed joint joint:left_shoulder_pitch_03
- removed joint joint:left_shoulder_roll_03
- removed joint joint:left_shoulder_yaw_02
- removed joint joint:left_wrist_02
- removed joint joint:leg0_(1):Fastened_1
- removed joint joint:leg0_(1):Fastened_2
- removed joint joint:leg0_(2):Fastened_1
- removed joint joint:leg0_(2):Fastened_2
- removed joint joint:leg1_(1):Fastened_1
- removed joint joint:leg1_(1):Fastened_2
- removed joint joint:leg2_(1):Fastened_1
- removed joint joint:leg2_(1):Fastened_2
- removed joint joint:leg2_(2):Fastened_1
- removed joint joint:leg2_(2):Fastened_2
- removed joint joint:leg3_(1):Fastened_2
- removed joint joint:leg3_(1):Fastened_3
- removed joint joint:leg3_(1):Fastened_4
- removed joint joint:leg3_(1):Fastened_5
- removed joint joint:right_ankle_02
- removed joint joint:right_elbow_02
- removed joint joint:right_hip_pitch_04
- removed joint joint:right_hip_roll_03
- removed joint joint:right_hip_yaw_03
- removed joint joint:right_knee_04
- removed joint joint:right_shoulder_pitch_03
- removed joint joint:right_shoulder_roll_03
- removed joint joint:right_shoulder_yaw_02
- removed joint joint:right_wrist_02
- added joint floating_base_joint: type fixed, parent floating_base_link, child body1_part, origin xyz=0 0 0 rpy=1.57 0.00 3.14
- added joint imu_link: type fixed, parent body1_part, child imu, origin xyz=0.039989 -0.127910 0 rpy=-1.570796 0 0
- added joint left_ankle_02: type revolute, parent leg3_shell1, child foot1, origin xyz=0 -0.300000 0.009500 rpy=0 0 0, axis 0 0 -1, limit lower=-0.698132 upper=0.698132 effort=17 velocity=12.566
- added joint left_elbow_02: type revolute, parent arm2_shell, child arm3_shell, origin xyz=-0.027000 0 -0.098000 rpy=-3.141593 -1.570796 0, axis 0 0 1, limit lower=-2.530727 upper=0 effort=17 velocity=12.566
- added joint left_hip_pitch_04: type revolute, parent body1_part, child leg0_shell, origin xyz=-0.000011 -0.432010 0.088700 rpy=-3.141593 0 -3.141593, axis 0 0 1, limit lower=-1.570796 upper=1.570796 effort=120 velocity=6.283
- added joint left_hip_roll_03: type revolute, parent leg0_shell, child leg1_shell, origin xyz=0.027500 0 -0.069500 rpy=-1.570796 0 1.570796, axis 0 0 1, limit lower=-3.185226 upper=0.349066 effort=60 velocity=6.283
- added joint left_hip_yaw_03: type revolute, parent leg1_shell, child leg2_shell, origin xyz=-0.157500 0.000120 0.027500 rpy=0 1.570796 0, axis 0 0 1, limit lower=-1.570796 upper=1.570796 effort=60 velocity=6.283
- added joint left_knee_04: type revolute, parent leg2_shell, child leg3_shell1, origin xyz=0 -0.027000 -0.142500 rpy=1.570796 0 0, axis 0 0 -1, limit lower=0 upper=2.094395 effort=120 velocity=6.283
- added joint left_shoulder_pitch_03: type revolute, parent body1_part, child shoulder, origin xyz=-0.000011 0.018090 0.188500 rpy=3.141593 0 3.141593, axis 0 0 1, limit lower=0 upper=3.141593 effort=60 velocity=6.283
- added joint left_shoulder_roll_03: type revolute, parent shoulder, child arm1_top, origin xyz=0.023512 0.000056 -0.067500 rpy=1.570796 0 1.570796, axis 0 0 -1, limit lower=-3.630285 upper=0.479966 effort=60 velocity=6.283
- added joint left_shoulder_yaw_02: type revolute, parent arm1_top, child arm2_shell, origin xyz=-0.140500 0 -0.023500 rpy=-1.570796 0 -1.570796, axis 0 0 1, limit lower=-1.570796 upper=1.570796 effort=17 velocity=12.566
- added joint left_wrist_02: type revolute, parent arm3_shell, child hand_shell, origin xyz=-0.182500 0 0.021500 rpy=-1.570796 0 -1.570796, axis 0 0 1, limit lower=-3.141593 upper=3.141593 effort=17 velocity=12.566
- added joint right_ankle_02: type revolute, parent leg3_shell11, child foot3, origin xyz=0 -0.300000 -0.035500 rpy=3.141593 0 3.141593, axis 0 0 1.0, limit lower=-0.698132 upper=0.698132 effort=17 velocity=12.566
- added joint right_elbow_02: type revolute, parent arm2_shell_2, child arm3_shell2, origin xyz=0 -0.027000 0.097500 rpy=-1.570796 1.570796 0, axis 0 0 1, limit lower=0 upper=2.530727 effort=17 velocity=12.566
- added joint right_hip_pitch_04: type revolute, parent body1_part, child leg0_shell_2, origin xyz=-0.000011 -0.432010 -0.089200 rpy=0 0 -3.141593, axis 0 0 1, limit lower=-1.570796 upper=1.570796 effort=120 velocity=6.283
- added joint right_hip_roll_03: type revolute, parent leg0_shell_2, child leg1_shell3, origin xyz=0.027500 0 -0.069000 rpy=1.570796 0 -1.570796, axis 0 0 1, limit lower=-0.349066 upper=3.185226 effort=60 velocity=6.283
- added joint right_hip_yaw_03: type revolute, parent leg1_shell3, child leg2_shell_2, origin xyz=-0.157500 -0.000120 0.027500 rpy=-3.141593 -1.570796 0, axis 0 0 1, limit lower=-1.570796 upper=1.570796 effort=60 velocity=6.283
- added joint right_knee_04: type revolute, parent leg2_shell_2, child leg3_shell11, origin xyz=0 -0.027000 -0.142500 rpy=1.570796 0 0, axis 0 0 -1, limit lower=-2.094395 upper=0 effort=120 velocity=6.283
- added joint right_shoulder_pitch_03: type revolute, parent body1_part, child shoulder_2, origin xyz=-0.000011 0.018090 -0.188500 rpy=0 0 -3.141593, axis 0 0 1, limit lower=-3.141593 upper=0 effort=60 velocity=6.283
- added joint right_shoulder_roll_03: type revolute, parent shoulder_2, child arm1_top_2, origin xyz=0.023512 -0.000056 -0.067500 rpy=1.570796 0 -1.570796, axis 0 0 1, limit lower=-0.479966 upper=3.630285 effort=60 velocity=6.283
- added joint right_shoulder_yaw_02: type revolute, parent arm1_top_2, child arm2_shell_2, origin xyz=-0.140500 0 0.022500 rpy=-3.141593 1.570796 0, axis 0 0 -1, limit lower=-1.570796 upper=1.570796 effort=17 velocity=12.566
- added joint right_wrist_02: type revolute, parent arm3_shell2, child hand_shell_2, origin xyz=-0.182500 0 0.021500 rpy=1.570796 0 1.570796, axis 0 0 1, limit lower=-3.141593 upper=3.141593 effort=17 velocity=12.566
