Commit message: update imu setup

File: imu_bench/robot.urdf (robot description, URDF)
Before this commit: robot assembly_1, 6 links, 5 joints
Links:
- removed link floating_base_link
- link Motor_Weight_Mount: mass 0.108000 -> 0.108; geometry collision mesh filename=meshes/Motor_Weight_Mount.stl; visual mesh filename=meshes/Motor_Weight_Mount.stl
- link STS3215: mass 0.341126 -> 0.34112575; geometry collision mesh filename=meshes/STS3215.stl; visual mesh filename=meshes/STS3215.stl
- link imu: mass 0.005700 -> 0.0057; geometry collision mesh filename=meshes/imu.stl; visual mesh filename=meshes/imu.stl
- link imu_2: mass 0.005700 -> 0.0057; geometry collision mesh filename=meshes/imu_2.stl; visual mesh filename=meshes/imu_2.stl
- link imu_3: mass 0.005700 -> 0.0057; geometry collision mesh filename=meshes/imu_3.stl; visual mesh filename=meshes/imu_3.stl
Joints:
- removed joint floating_base_joint
- joint dof_servo_out: limit lower=-1.570796 upper=1.570796 effort=5 velocity=6.28 -> lower=-1.5707963 upper=1.5707963 effort=5 velocity=6.28; origin xyz=0.000007 -0.010299 0.088440 rpy=-1.570796 0 0 -> xyz=7.4096296e-06 -0.010298954 0.088439782 rpy=-1.5707963 0 0
- joint fix_imu_bottom: origin xyz=0.017732 -0.003224 -0.067900 rpy=3.141593 0 3.141593 -> xyz=0.017731837 -0.0032239537 -0.067899562 rpy=3.1415927 0 3.1415927
- joint fix_imu_front_side: origin xyz=0.000007 -0.029724 -0.041560 rpy=1.570796 1.570796 0 -> xyz=7.4096296e-06 -0.029723954 -0.041560218 rpy=1.5707963 1.5707963 0
- joint fix_imu_right_side: origin xyz=0.020007 -0.003224 -0.023810 rpy=0 1.570796 0 -> xyz=0.02000741 -0.0032239537 -0.023810218 rpy=0 1.5707963 0

Commit message: fixes with choosing base link

File: imu_bench/robot.urdf (robot description, URDF)
Before this commit: robot assembly_1, 5 links, 4 joints
Links:
- added link floating_base_link, mass 0.001; visual sphere radius=0.01
- link Motor_Weight_Mount: mass 0.108 -> 0.092000; geometry collision mesh filename=meshes/Motor_Weight_Mount.collision.stl; visual mesh filename=meshes/Motor_Weight_Mount.stl
- link STS3215: mass 0.34112575 -> 0.270643; geometry collision mesh filename=meshes/STS3215.collision.stl; visual mesh filename=meshes/STS3215.stl
- link imu: mass 0.0057 -> 0.005700; geometry collision mesh filename=meshes/imu.collision.stl; visual mesh filename=meshes/imu.stl
- link imu_2: mass 0.0057 -> 0.005700; geometry collision mesh filename=meshes/imu_2.collision.stl; visual mesh filename=meshes/imu_2.stl
- link imu_3: mass 0.0057 -> 0.005700; geometry collision mesh filename=meshes/imu_3.collision.stl; visual mesh filename=meshes/imu_3.stl
Joints:
- removed joint dof_servo_out
- removed joint fix_imu_bottom
- removed joint fix_imu_front_side
- removed joint fix_imu_right_side
- added joint floating_base_joint: type fixed, parent floating_base_link, child STS3215, origin xyz=0 0 0 rpy=0.00 -1.57 0.00
- added joint imu_bottom: type fixed, parent Motor_Weight_Mount, child imu_3, origin xyz=-0.156339 0 -0.042875 rpy=1.570796 0 -1.570796
- added joint imu_front_side: type fixed, parent Motor_Weight_Mount, child imu, origin xyz=-0.130000 0 -0.057375 rpy=3.141593 0 3.141593
- added joint imu_right_side: type fixed, parent Motor_Weight_Mount, child imu_2, origin xyz=-0.130000 0.020000 -0.042875 rpy=1.570796 0 3.141593
- added joint servo_out: type revolute, parent STS3215, child Motor_Weight_Mount, origin xyz=-0.011909 -0.000014 -0.020256 rpy=3.141593 0 0, axis 0 0 -1, limit lower=-1.570796 upper=1.570796 effort=5 velocity=6.28
