Commit message: painful up-rev non-automated mjcfs

File: kbot-v2-feet/robot.urdf (robot description, URDF)
Before this commit: robot kbotv2p0_nohands, 113 links, 106 joints
Links:
- removed link link:7inlcd_(1)
- removed link link:BATT-SLOT_(1)
- removed link link:Battery_Back_Case_(1)
- removed link link:Battery_CellPack_(1)
- removed link link:Battery_Cover_(1)
- removed link link:Battery_Handle_(1)
- removed link link:Battery_Middle_Cover_(1)
- removed link link:Battery_Plate_(1)
- removed link link:Bearing_(1)
- removed link link:Bearing_(2)
- removed link link:Comp_Holder_(1)
- removed link link:Flat_Foot_Pad_Left_(1)
- removed link link:Flat_Foot_Pad_Right_(1)
- removed link link:KB-C-501X_Left_Bayonet_Adapter_Hard_Stop_(1)
- removed link link:KB-C-501X_Right_Bayonet_Adapter_Hard_Stop_(1)
- removed link link:KB-D-501L_L_LEG-FOOT_(1)
- removed link link:KB-D-501R_R_LEG-FOOT_(1)
- removed link link:KB-D-502L_ANKLE-SHAFT_vis_(1)
- removed link link:KB-D-502R_ANKLE-SHAFT_vis_(1)
- removed link link:KB-D-503X_ANKLE_LINK-S-LEFT_vis_(1)
- removed link link:KB-D-503X_ANKLE_LINK-S-RIGHT_vis_(1)
- removed link link:KB-D-504X_BOLT_ANKLE_L_vis_(1)
- removed link link:KB-D-504X_BOLT_ANKLE_R_vis_(1)
- removed link link:KC-C-101L_ShldYokeDrive_(2)
- removed link link:KC-C-101R_ShldYokeDrive_(1)
- removed link link:KC-C-102L_ShldYokeIdle_(1)
- removed link link:KC-C-102R_ShldYokeIdle_(1)
- removed link link:KC-C-103L_PitchHardstopStatic_(1)
- removed link link:KC-C-103R_PitchHardstopStatic_(1)
- removed link link:KC-C-104L_PitchHardstopDriven_(1)
- removed link link:KC-C-104R_PitchHardstopDriven_(1)
- removed link link:KC-C-105X_ShldYokeBearingPin_(1)
- removed link link:KC-C-105X_ShldYokeBearingPin_(2)
- removed link link:KC-C-201L_(2)
- removed link link:KC-C-201L_UpBicepDrive_(2)
- removed link link:KC-C-201R_(1)
- removed link link:KC-C-201R_UpBicepDrive_(1)
- removed link link:KC-C-202L_(1)
- removed link link:KC-C-202L_UpBicepIdle_(1)
- removed link link:KC-C-202R_(1)
- removed link link:KC-C-202R_UpBicepIdle_(1)
- removed link link:KC-C-203X_(1)
- removed link link:KC-C-203X_(2)
- removed link link:KC-C-401L_L_UpForearmDrive_(1)
- removed link link:KC-C-401R_R_UpForearmDrive_(1)
- removed link link:KC-C-402L_Forearm_Upper_Idle_(2)
- removed link link:KC-C-402R_Forearm_Upper_Idle_(1)
- removed link link:KC-D-101L_L_Hip_Static_(1)
- removed link link:KC-D-101R_R_Hip_Static_(1)
- removed link link:KC-D-102L_L_Hip_Yoke_Drive_(1)
- removed link link:KC-D-102R_R_Hip_Yoke_Drive_(1)
- removed link link:KC-D-103L_L_Hip_Yoke_Idle_(1)
- removed link link:KC-D-103R_R_Hip_Yoke_Idle_(1)
- removed link link:KC-D-104R_Hip_Yoke_Hardstop_vis_(1)
- removed link link:KC-D-104_L_Hip_Yoke_Hardstop_vis_(1)
- removed link link:KC-D-105L_HipYokeHardstopTooth_vis_(1)
- removed link link:KC-D-105R_HipYokeHardstopTooth_vis_(1)
- removed link link:KC-D-106X_Hip_Bearing_Pin_L_vis_(1)
- removed link link:KC-D-106X_Hip_Bearing_Pin_R_vis_(1)
- removed link link:KC-D-107L_L_Cover_(1)
- removed link link:KC-D-107R_R_Cover_(1)
- removed link link:KC-D-201L_UpperThigh_Act_(1)
- removed link link:KC-D-201L_UpperThigh_Idle_(1)
- removed link link:KC-D-201R_UpperThigh_Act_(1)
- removed link link:KC-D-201R_UpperThigh_Idle_(1)
- removed link link:KC-D-203L_Thigh_Roll_Hardstop_vis_(1)
- removed link link:KC-D-203R_Thigh_Roll_Hardstop_vis_(1)
- removed link link:KC-D-301L_L_Femur_Lower_Drive_(1)
- removed link link:KC-D-301R_R_Femur_Lower_Drive_(1)
- removed link link:KC-D-302L_L_Femur_Lower_Idle_(1)
- removed link link:KC-D-302R_Femur_Lower_Idle_(1)
- removed link link:KC-D-401L_L_Shin_Drive_(1)
- removed link link:KC-D-401R_R_Shin_Drive_(1)
- removed link link:KC-D-402L_L_Shin_Idle_(1)
- removed link link:KC-D-402R_R_Shin_Idle_(1)
- removed link link:KC-D-403L_LEG-SHIN_COVER_vis_(1)
- removed link link:KC-D-403R_LEG-SHIN_COVER_vis_(1)
- removed link link:KC-D-506L_EndStop_80deg_vis_(1)
- removed link link:KC-D-506R_EndStop_80deg_vis_(1)
- removed link link:LOCKED_Middle_Cover_(1)
- removed link link:RS00_(1)
- removed link link:RS00_(2)
- removed link link:RS02_(1)
- removed link link:RS02_(2)
- removed link link:RS02_(3)
- removed link link:RS02_(4)
- removed link link:RS02_(5)
- removed link link:RS02_(6)
- removed link link:RS03_(1)
- removed link link:RS03_(2)
- removed link link:RS03_(3)
- removed link link:RS03_(4)
- removed link link:RS03_(5)
- removed link link:RS03_(6)
- removed link link:RS03_(7)
- removed link link:RS03_(8)
- removed link link:RS04_(1)
- removed link link:RS04_(2)
- removed link link:RS04_(3)
- removed link link:RS04_(4)
- removed link link:Torso-top_(1)
- removed link link:Torso_Bottom_(1)
- removed link link:Torso_Inside_(1)
- removed link link:Torso_Side_Cover_Left_(1)
- removed link link:Torso_Side_Cover_Right_(1)
- removed link link:Torso_Side_Left_(1)
- removed link link:Torso_Side_Right_(1)
- removed link link:front_bottom_cover_(1)
- removed link link:front_cover_(1)
- removed link link:head_back_(1)
- removed link link:imu_(1)
- removed link link:top_cover_(1)
- removed link link:torso-front-up_(1)
- added link KB_C_501X_Left_Bayonet_Adapter_Hard_Stop, mass 0.152198; visual mesh filename=meshes/KB_C_501X_Left_Bayonet_Adapter_Hard_Stop.stl
- added link KB_C_501X_Right_Bayonet_Adapter_Hard_Stop, mass 0.152198; visual mesh filename=meshes/KB_C_501X_Right_Bayonet_Adapter_Hard_Stop.stl
- added link KB_D_501L_L_LEG_FOOT, mass 0.483858; collision mesh filename=meshes/KB_D_501L_L_LEG_FOOT.collision.stl; visual mesh filename=meshes/KB_D_501L_L_LEG_FOOT.stl
- added link KB_D_501R_R_LEG_FOOT, mass 0.483858; collision mesh filename=meshes/KB_D_501R_R_LEG_FOOT.collision.stl; visual mesh filename=meshes/KB_D_501R_R_LEG_FOOT.stl
- added link KC_C_104L_PitchHardstopDriven, mass 0.584843; visual mesh filename=meshes/KC_C_104L_PitchHardstopDriven.stl
- added link KC_C_104R_PitchHardstopDriven, mass 0.584848; visual mesh filename=meshes/KC_C_104R_PitchHardstopDriven.stl
- added link KC_C_202L, mass 0.579259; visual mesh filename=meshes/KC_C_202L.stl
- added link KC_C_202R, mass 0.743508; visual mesh filename=meshes/KC_C_202R.stl
- added link KC_C_401L_L_UpForearmDrive, mass 0.585219; visual mesh filename=meshes/KC_C_401L_L_UpForearmDrive.stl
- added link KC_C_401R_R_UpForearmDrive, mass 0.585204; visual mesh filename=meshes/KC_C_401R_R_UpForearmDrive.stl
- added link KC_D_102L_L_Hip_Yoke_Drive, mass 0.530424; visual mesh filename=meshes/KC_D_102L_L_Hip_Yoke_Drive.stl
- added link KC_D_102R_R_Hip_Yoke_Drive, mass 0.530428; visual mesh filename=meshes/KC_D_102R_R_Hip_Yoke_Drive.stl
- added link KC_D_301L_L_Femur_Lower_Drive, mass 2.343629; visual mesh filename=meshes/KC_D_301L_L_Femur_Lower_Drive.stl
- added link KC_D_301R_R_Femur_Lower_Drive, mass 2.343635; visual mesh filename=meshes/KC_D_301R_R_Femur_Lower_Drive.stl
- added link KC_D_401L_L_Shin_Drive, mass 1.670535; visual mesh filename=meshes/KC_D_401L_L_Shin_Drive.stl
- added link KC_D_401R_R_Shin_Drive, mass 1.670592; visual mesh filename=meshes/KC_D_401R_R_Shin_Drive.stl
- added link RS03_3, mass 1.676509; visual mesh filename=meshes/RS03_3.stl
- added link RS03_4, mass 2.373184; visual mesh filename=meshes/RS03_4.stl
- added link RS03_5, mass 2.373239; visual mesh filename=meshes/RS03_5.stl
- added link RS03_6, mass 1.676479; visual mesh filename=meshes/RS03_6.stl
- added link Torso_Side_Right, mass 13.322034; visual mesh filename=meshes/Torso_Side_Right.stl
- added link floating_base_link, mass 0.001; visual sphere radius=0.01
- added link imu, mass 0.005700; visual mesh filename=meshes/imu.stl
Joints:
- removed joint joint:dof_back_top
- removed joint joint:dof_batt_2slot
- removed joint joint:dof_batt_slot
- removed joint joint:dof_btm
- removed joint joint:dof_comp_holder
- removed joint joint:dof_feet_pad_left
- removed joint joint:dof_feet_pad_right
- removed joint joint:dof_front_btm
- removed joint joint:dof_front_head
- removed joint joint:dof_front_panel
- removed joint joint:dof_front_top
- removed joint joint:dof_head_fix
- removed joint joint:dof_hiproll_upperthigh_left
- removed joint joint:dof_hiproll_upperthigh_right
- removed joint joint:dof_hipyaw_upperthigh_left
- removed joint joint:dof_hipyaw_upperthigh_right
- removed joint joint:dof_hipyoke_left
- removed joint joint:dof_hipyoke_right
- removed joint joint:dof_lcd
- removed joint joint:dof_left_ankle_02
- removed joint joint:dof_left_anklemotor
- removed joint joint:dof_left_bicepyaw02
- removed joint joint:dof_left_elbow02fix
- removed joint joint:dof_left_elbow_02
- removed joint joint:dof_left_fixshldr03
- removed joint joint:dof_left_forearm_idle
- removed joint joint:dof_left_hip
- removed joint joint:dof_left_hip_idle
- removed joint joint:dof_left_hip_pitch_04
- removed joint joint:dof_left_hip_roll_03
- removed joint joint:dof_left_hip_yaw_03
- removed joint joint:dof_left_idleShlr
- removed joint joint:dof_left_knee_04
- removed joint joint:dof_left_lowerbicep_idle
- removed joint joint:dof_left_rs03
- removed joint joint:dof_left_shldr
- removed joint joint:dof_left_shoulder_pitch_03
- removed joint joint:dof_left_shoulder_roll_03
- removed joint joint:dof_left_shoulder_yaw_02
- removed joint joint:dof_left_torso
- removed joint joint:dof_left_upper_bicep_idle
- removed joint joint:dof_left_wrist_00
- removed joint joint:dof_lower_thigh_drive_left
- removed joint joint:dof_lower_thigh_drive_right
- removed joint joint:dof_lower_thigh_idle_left
- removed joint joint:dof_mid_head
- removed joint joint:dof_right_ankle_02
- removed joint joint:dof_right_anklemotor
- removed joint joint:dof_right_bicepyaw_02
- removed joint joint:dof_right_elbow02fix
- removed joint joint:dof_right_elbow_02
- removed joint joint:dof_right_fixshldr03
- removed joint joint:dof_right_forearm_idle
- removed joint joint:dof_right_hip
- removed joint joint:dof_right_hip_idle
- removed joint joint:dof_right_hip_pitch_04
- removed joint joint:dof_right_hip_roll_03
- removed joint joint:dof_right_hip_yaw_03
- removed joint joint:dof_right_idleShlr
- removed joint joint:dof_right_knee_04
- removed joint joint:dof_right_lowerbicep_idle
- removed joint joint:dof_right_rs03
- removed joint joint:dof_right_shldr
- removed joint joint:dof_right_shoulder_pitch_03
- removed joint joint:dof_right_shoulder_roll_03
- removed joint joint:dof_right_shoulder_yaw_02
- removed joint joint:dof_right_upper_bicep_idle
- removed joint joint:dof_right_wrist00fix
- removed joint joint:dof_right_wrist_00
- removed joint joint:dof_shin_shells_left
- removed joint joint:dof_shin_shells_right
- removed joint joint:dof_top_torso
- removed joint joint:dof_upperthigh_shell_left
- removed joint joint:dof_upperthigh_shell_right
- removed joint joint:doft_left_wrist00fix
- removed joint joint:fix_ankle_bolt_left
- removed joint joint:fix_ankle_bolt_right
- removed joint joint:fix_ankle_motor
- removed joint joint:fix_ankle_motor2
- removed joint joint:fix_ankle_motor3
- removed joint joint:fix_hipyoke_pin_left
- removed joint joint:fix_hipyoke_pin_right
- removed joint joint:fix_left_hipyaw_hardstop_vis
- removed joint joint:fix_left_yaw_hardstop_vis
- removed joint joint:fix_lefthippitch_hardstop
- removed joint joint:fix_lefthippitch_hardstop2_vis
- removed joint joint:fix_right_hipyaw_hardstop_vis
- removed joint joint:fix_right_yaw_hardstop_vis
- removed joint joint:fix_righthippitch_hardstop
- removed joint joint:fix_righthippitch_hardstop2_vis
- removed joint joint:fixed_batt1
- removed joint joint:fixed_batt2
- removed joint joint:fixed_batt3
- removed joint joint:fixed_battFront
- removed joint joint:fixed_battHandle
- removed joint joint:fixed_knee_idle_left
- removed joint joint:fixed_knee_idle_right
- removed joint joint:fixed_left03_hrdstop
- removed joint joint:fixed_left_Shldrbearing1
- removed joint joint:fixed_left_Shldrhrdstp
- removed joint joint:fixed_left_shldrbearing2
- removed joint joint:fixed_right03_hrdstop
- removed joint joint:fixed_right_Shldrbearing1
- removed joint joint:fixed_right_Shldrbearing2
- removed joint joint:fixed_right_Shldrhrdstp
- removed joint joint:frame_imu_site
- added joint dof_left_ankle_02: type revolute, parent KC_D_401L_L_Shin_Drive, child KB_D_501L_L_LEG_FOOT, origin xyz=-0.030000 -0.290000 0.035100 rpy=-3.141593 0 0, axis 0 0 -1, limit lower=-0.785398 upper=0.296706 effort=17 velocity=12.566
- added joint dof_left_elbow_02: type revolute, parent KC_C_202L, child KC_C_401L_L_UpForearmDrive, origin xyz=-0.018500 0.010000 0.137000 rpy=-3.141593 1.570796 0, axis 0 0 -1, limit lower=-2.478368 upper=0 effort=17 velocity=12.566
- added joint dof_left_hip_pitch_04: type revolute, parent Torso_Side_Right, child KC_D_102L_L_Hip_Yoke_Drive, origin xyz=0.147969 0.000007 -0.284479 rpy=-1.570796 0 1.570796, axis 0 0 1, limit lower=-1.047198 upper=2.216568 effort=120 velocity=6.283
- added joint dof_left_hip_roll_03: type revolute, parent KC_D_102L_L_Hip_Yoke_Drive, child RS03_5, origin xyz=-0.028250 0.030000 -0.071000 rpy=0 1.570796 0, axis 0 0 -1, limit lower=-0.209440 upper=2.268928 effort=60 velocity=6.283
- added joint dof_left_hip_yaw_03: type revolute, parent RS03_5, child KC_D_301L_L_Femur_Lower_Drive, origin xyz=0 0.143000 0.024250 rpy=-1.570796 0 0, axis 0 0 -1, limit lower=-1.570796 upper=1.570796 effort=60 velocity=6.283
- added joint dof_left_knee_04: type revolute, parent KC_D_301L_L_Femur_Lower_Drive, child KC_D_401L_L_Shin_Drive, origin xyz=-0.020500 -0.021000 0.212000 rpy=-1.570796 0 -1.570796, axis 0 0 1, limit lower=0 upper=2.705260 effort=120 velocity=6.283
- added joint dof_left_shoulder_pitch_03: type revolute, parent Torso_Side_Right, child KC_C_104L_PitchHardstopDriven, origin xyz=0.213969 0.000007 0.126021 rpy=-1.570796 0 1.570796, axis 0 0 1, limit lower=-1.047198 upper=3.490658 effort=60 velocity=6.283
- added joint dof_left_shoulder_roll_03: type revolute, parent KC_C_104L_PitchHardstopDriven, child RS03_6, origin xyz=-0.024250 0 -0.080000 rpy=-3.141593 1.570796 0, axis 0 0 1, limit lower=-0.383972 upper=1.658063 effort=60 velocity=6.283
- added joint dof_left_shoulder_yaw_02: type revolute, parent RS03_6, child KC_C_202L, origin xyz=0.013000 -0.142000 -0.030250 rpy=1.570796 0 0, axis 0 0 -1, limit lower=-1.658063 upper=1.658063 effort=17 velocity=12.566
- added joint dof_left_wrist_00: type revolute, parent KC_C_401L_L_UpForearmDrive, child KB_C_501X_Left_Bayonet_Adapter_Hard_Stop, origin xyz=-0.103000 0.017350 -0.018000 rpy=-3.141593 1.570796 0, axis 0 0 -1, limit lower=-1.745329 upper=1.745329 effort=14 velocity=12.566
- added joint dof_right_ankle_02: type revolute, parent KC_D_401R_R_Shin_Drive, child KB_D_501R_R_LEG_FOOT, origin xyz=-0.030000 0.290000 0.035100 rpy=0 0 0, axis 0 0 1, limit lower=-0.296706 upper=0.785398 effort=17 velocity=12.566
- added joint dof_right_elbow_02: type revolute, parent KC_C_202R, child KC_C_401R_R_UpForearmDrive, origin xyz=0.018500 -0.010000 -0.137000 rpy=0 1.570796 0, axis 0 0 -1, limit lower=0 upper=2.478368 effort=17 velocity=12.566
- added joint dof_right_hip_pitch_04: type revolute, parent Torso_Side_Right, child KC_D_102R_R_Hip_Yoke_Drive, origin xyz=0.037469 0.000007 -0.284479 rpy=1.570796 0 1.570796, axis 0 0 1, limit lower=-2.216568 upper=1.047198 effort=120 velocity=6.283
- added joint dof_right_hip_roll_03: type revolute, parent KC_D_102R_R_Hip_Yoke_Drive, child RS03_4, origin xyz=-0.028250 -0.030000 -0.071000 rpy=3.141593 -1.570796 0, axis 0 0 -1, limit lower=-2.268928 upper=0.209440 effort=60 velocity=6.283
- added joint dof_right_hip_yaw_03: type revolute, parent RS03_4, child KC_D_301R_R_Femur_Lower_Drive, origin xyz=0 0.143000 0.024250 rpy=-1.570796 0 0, axis 0 0 -1, limit lower=-1.570796 upper=1.570796 effort=60 velocity=6.283
- added joint dof_right_knee_04: type revolute, parent KC_D_301R_R_Femur_Lower_Drive, child KC_D_401R_R_Shin_Drive, origin xyz=0.020500 -0.021000 0.212000 rpy=1.570796 0 -1.570796, axis 0 0 1, limit lower=-2.705260 upper=0 effort=120 velocity=6.283
- added joint dof_right_shoulder_pitch_03: type revolute, parent Torso_Side_Right, child KC_C_104R_PitchHardstopDriven, origin xyz=-0.028031 0.000007 0.126021 rpy=1.570796 0 1.570796, axis 0 0 1, limit lower=-2.617994 upper=2.094395 effort=60 velocity=6.283
- added joint dof_right_shoulder_roll_03: type revolute, parent KC_C_104R_PitchHardstopDriven, child RS03_3, origin xyz=-0.024250 0 -0.080000 rpy=-3.141593 -1.570796 0, axis 0 0 -1, limit lower=-1.658063 upper=0.383972 effort=60 velocity=6.283
- added joint dof_right_shoulder_yaw_02: type revolute, parent RS03_3, child KC_C_202R, origin xyz=-0.013000 0.142000 0.030250 rpy=1.570796 0 0, axis 0 0 1, limit lower=-1.658063 upper=1.658063 effort=17 velocity=12.566
- added joint dof_right_wrist_00: type revolute, parent KC_C_401R_R_UpForearmDrive, child KB_C_501X_Right_Bayonet_Adapter_Hard_Stop, origin xyz=0.103000 0.017350 -0.018000 rpy=0 -1.570796 0, axis 0 0 1, limit lower=-1.745329 upper=1.745329 effort=14 velocity=12.566
- added joint floating_base_joint: type fixed, parent floating_base_link, child Torso_Side_Right, origin xyz=0 0 0 rpy=0.00 0.00 1.57
- added joint frame_imu_site: type fixed, parent Torso_Side_Right, child imu, origin xyz=0.121783 0.043292 0.231518 rpy=1.582557 1.570794 1.582557
