Commit message: Remove the heavy K-Bot V2 from URDFs and K-Scale assets  (#32)
* fixes

* add back files

* add back kbot-v1-feet files

* painful up-rev non-automated mjcfs

File: kbot-v2-feet/robot.urdf (robot description, URDF)
Before this commit: robot kbot-v2, 22 links, 21 joints
Links:
- removed link KB_B_102B_TORSO_BOTTOM
- removed link KB_C_501X_Bayonet_Adapter_Hard_Stop
- removed link KB_C_501X_Bayonet_Adapter_Hard_Stop_2
- removed link KB_D_102L_L_Hip_Yoke_Drive
- removed link KB_D_102R_R_Hip_Yoke_Drive
- removed link KB_D_301L_L_Femur_Lower_Drive
- removed link KB_D_301R_R_Femur_Lower_Drive
- removed link KB_D_401R_R_Shin_Drive
- removed link KB_D_402L_L_Shin_Idle
- removed link L_Bicep_Lower_Drive
- removed link L_Forearm_Upper_Drive
- removed link R_Bicep_Lower_Drive
- removed link R_Forearm_Upper_Structural
- removed link YOKE_STOP_INNER
- removed link YOKE_STOP_INNER_2
- added link KB_C_501X_Left_Bayonet_Adapter_Hard_Stop, mass 0.152198; visual mesh filename=meshes/KB_C_501X_Left_Bayonet_Adapter_Hard_Stop.stl
- added link KB_C_501X_Right_Bayonet_Adapter_Hard_Stop, mass 0.152198; visual mesh filename=meshes/KB_C_501X_Right_Bayonet_Adapter_Hard_Stop.stl
- added link KC_C_104L_PitchHardstopDriven, mass 0.584843; visual mesh filename=meshes/KC_C_104L_PitchHardstopDriven.stl
- added link KC_C_104R_PitchHardstopDriven, mass 0.584848; visual mesh filename=meshes/KC_C_104R_PitchHardstopDriven.stl
- added link KC_C_202L, mass 0.579259; visual mesh filename=meshes/KC_C_202L.stl
- added link KC_C_202R, mass 0.743508; visual mesh filename=meshes/KC_C_202R.stl
- added link KC_C_401L_L_UpForearmDrive, mass 0.585219; visual mesh filename=meshes/KC_C_401L_L_UpForearmDrive.stl
- added link KC_C_401R_R_UpForearmDrive, mass 0.585204; visual mesh filename=meshes/KC_C_401R_R_UpForearmDrive.stl
- added link KC_D_102L_L_Hip_Yoke_Drive, mass 0.530424; visual mesh filename=meshes/KC_D_102L_L_Hip_Yoke_Drive.stl
- added link KC_D_102R_R_Hip_Yoke_Drive, mass 0.530428; visual mesh filename=meshes/KC_D_102R_R_Hip_Yoke_Drive.stl
- added link KC_D_301L_L_Femur_Lower_Drive, mass 2.343629; visual mesh filename=meshes/KC_D_301L_L_Femur_Lower_Drive.stl
- added link KC_D_301R_R_Femur_Lower_Drive, mass 2.343635; visual mesh filename=meshes/KC_D_301R_R_Femur_Lower_Drive.stl
- added link KC_D_401L_L_Shin_Drive, mass 1.670535; visual mesh filename=meshes/KC_D_401L_L_Shin_Drive.stl
- added link KC_D_401R_R_Shin_Drive, mass 1.670592; visual mesh filename=meshes/KC_D_401R_R_Shin_Drive.stl
- added link Torso_Side_Right, mass 13.322034; visual mesh filename=meshes/Torso_Side_Right.stl
- added link imu, mass 0.005700; visual mesh filename=meshes/imu.stl
- link KB_D_501L_L_LEG_FOOT: mass 0.492748 -> 0.483858; geometry collision mesh filename=meshes/KB_D_501L_L_LEG_FOOT.collision.stl; visual mesh filename=meshes/KB_D_501L_L_LEG_FOOT.stl
- link KB_D_501R_R_LEG_FOOT: mass 0.492747 -> 0.483858; geometry collision mesh filename=meshes/KB_D_501R_R_LEG_FOOT.collision.stl; visual mesh filename=meshes/KB_D_501R_R_LEG_FOOT.stl
- link RS03_3: mass 2.590316 -> 1.676509; geometry visual mesh filename=meshes/RS03_3.stl
- link RS03_4: mass 2.590429 -> 2.373184; geometry visual mesh filename=meshes/RS03_4.stl
- link RS03_5: mass 1.888573 -> 2.373239; geometry visual mesh filename=meshes/RS03_5.stl
- link RS03_6: mass 1.888599 -> 1.676479; geometry visual mesh filename=meshes/RS03_6.stl
Joints:
- removed joint left_ankle_02
- removed joint left_elbow_02
- removed joint left_hip_pitch_04
- removed joint left_hip_roll_03
- removed joint left_hip_yaw_03
- removed joint left_knee_04
- removed joint left_shoulder_pitch_03
- removed joint left_shoulder_roll_03
- removed joint left_shoulder_yaw_02
- removed joint left_wrist_02
- removed joint right_ankle_02
- removed joint right_elbow_02
- removed joint right_hip_pitch_04
- removed joint right_hip_roll_03
- removed joint right_hip_yaw_03
- removed joint right_knee_04
- removed joint right_shoulder_pitch_03
- removed joint right_shoulder_roll_03
- removed joint right_shoulder_yaw_02
- removed joint right_wrist_02
- added joint dof_left_ankle_02: type revolute, parent KC_D_401L_L_Shin_Drive, child KB_D_501L_L_LEG_FOOT, origin xyz=-0.030000 -0.290000 0.035100 rpy=-3.141593 0 0, axis 0 0 -1, limit lower=-0.785398 upper=0.296706 effort=17 velocity=12.566
- added joint dof_left_elbow_02: type revolute, parent KC_C_202L, child KC_C_401L_L_UpForearmDrive, origin xyz=-0.018500 0.010000 0.137000 rpy=-3.141593 1.570796 0, axis 0 0 -1, limit lower=-2.478368 upper=0 effort=17 velocity=12.566
- added joint dof_left_hip_pitch_04: type revolute, parent Torso_Side_Right, child KC_D_102L_L_Hip_Yoke_Drive, origin xyz=0.147969 0.000007 -0.284479 rpy=-1.570796 0 1.570796, axis 0 0 1, limit lower=-1.047198 upper=2.216568 effort=120 velocity=6.283
- added joint dof_left_hip_roll_03: type revolute, parent KC_D_102L_L_Hip_Yoke_Drive, child RS03_5, origin xyz=-0.028250 0.030000 -0.071000 rpy=0 1.570796 0, axis 0 0 -1, limit lower=-0.209440 upper=2.268928 effort=60 velocity=6.283
- added joint dof_left_hip_yaw_03: type revolute, parent RS03_5, child KC_D_301L_L_Femur_Lower_Drive, origin xyz=0 0.143000 0.024250 rpy=-1.570796 0 0, axis 0 0 -1, limit lower=-1.570796 upper=1.570796 effort=60 velocity=6.283
- added joint dof_left_knee_04: type revolute, parent KC_D_301L_L_Femur_Lower_Drive, child KC_D_401L_L_Shin_Drive, origin xyz=-0.020500 -0.021000 0.212000 rpy=-1.570796 0 -1.570796, axis 0 0 1, limit lower=0 upper=2.705260 effort=120 velocity=6.283
- added joint dof_left_shoulder_pitch_03: type revolute, parent Torso_Side_Right, child KC_C_104L_PitchHardstopDriven, origin xyz=0.213969 0.000007 0.126021 rpy=-1.570796 0 1.570796, axis 0 0 1, limit lower=-1.047198 upper=3.490658 effort=60 velocity=6.283
- added joint dof_left_shoulder_roll_03: type revolute, parent KC_C_104L_PitchHardstopDriven, child RS03_6, origin xyz=-0.024250 0 -0.080000 rpy=-3.141593 1.570796 0, axis 0 0 1, limit lower=-0.383972 upper=1.658063 effort=60 velocity=6.283
- added joint dof_left_shoulder_yaw_02: type revolute, parent RS03_6, child KC_C_202L, origin xyz=0.013000 -0.142000 -0.030250 rpy=1.570796 0 0, axis 0 0 -1, limit lower=-1.658063 upper=1.658063 effort=17 velocity=12.566
- added joint dof_left_wrist_00: type revolute, parent KC_C_401L_L_UpForearmDrive, child KB_C_501X_Left_Bayonet_Adapter_Hard_Stop, origin xyz=-0.103000 0.017350 -0.018000 rpy=-3.141593 1.570796 0, axis 0 0 -1, limit lower=-1.745329 upper=1.745329 effort=14 velocity=12.566
- added joint dof_right_ankle_02: type revolute, parent KC_D_401R_R_Shin_Drive, child KB_D_501R_R_LEG_FOOT, origin xyz=-0.030000 0.290000 0.035100 rpy=0 0 0, axis 0 0 1, limit lower=-0.296706 upper=0.785398 effort=17 velocity=12.566
- added joint dof_right_elbow_02: type revolute, parent KC_C_202R, child KC_C_401R_R_UpForearmDrive, origin xyz=0.018500 -0.010000 -0.137000 rpy=0 1.570796 0, axis 0 0 -1, limit lower=0 upper=2.478368 effort=17 velocity=12.566
- added joint dof_right_hip_pitch_04: type revolute, parent Torso_Side_Right, child KC_D_102R_R_Hip_Yoke_Drive, origin xyz=0.037469 0.000007 -0.284479 rpy=1.570796 0 1.570796, axis 0 0 1, limit lower=-2.216568 upper=1.047198 effort=120 velocity=6.283
- added joint dof_right_hip_roll_03: type revolute, parent KC_D_102R_R_Hip_Yoke_Drive, child RS03_4, origin xyz=-0.028250 -0.030000 -0.071000 rpy=3.141593 -1.570796 0, axis 0 0 -1, limit lower=-2.268928 upper=0.209440 effort=60 velocity=6.283
- added joint dof_right_hip_yaw_03: type revolute, parent RS03_4, child KC_D_301R_R_Femur_Lower_Drive, origin xyz=0 0.143000 0.024250 rpy=-1.570796 0 0, axis 0 0 -1, limit lower=-1.570796 upper=1.570796 effort=60 velocity=6.283
- added joint dof_right_knee_04: type revolute, parent KC_D_301R_R_Femur_Lower_Drive, child KC_D_401R_R_Shin_Drive, origin xyz=0.020500 -0.021000 0.212000 rpy=1.570796 0 -1.570796, axis 0 0 1, limit lower=-2.705260 upper=0 effort=120 velocity=6.283
- added joint dof_right_shoulder_pitch_03: type revolute, parent Torso_Side_Right, child KC_C_104R_PitchHardstopDriven, origin xyz=-0.028031 0.000007 0.126021 rpy=1.570796 0 1.570796, axis 0 0 1, limit lower=-2.617994 upper=2.094395 effort=60 velocity=6.283
- added joint dof_right_shoulder_roll_03: type revolute, parent KC_C_104R_PitchHardstopDriven, child RS03_3, origin xyz=-0.024250 0 -0.080000 rpy=-3.141593 -1.570796 0, axis 0 0 -1, limit lower=-1.658063 upper=0.383972 effort=60 velocity=6.283
- added joint dof_right_shoulder_yaw_02: type revolute, parent RS03_3, child KC_C_202R, origin xyz=-0.013000 0.142000 0.030250 rpy=1.570796 0 0, axis 0 0 1, limit lower=-1.658063 upper=1.658063 effort=17 velocity=12.566
- added joint dof_right_wrist_00: type revolute, parent KC_C_401R_R_UpForearmDrive, child KB_C_501X_Right_Bayonet_Adapter_Hard_Stop, origin xyz=0.103000 0.017350 -0.018000 rpy=0 -1.570796 0, axis 0 0 1, limit lower=-1.745329 upper=1.745329 effort=14 velocity=12.566
- added joint frame_imu_site: type fixed, parent Torso_Side_Right, child imu, origin xyz=0.121783 0.043292 0.231518 rpy=1.582557 1.570794 1.582557
- joint floating_base_joint: child KB_B_102B_TORSO_BOTTOM -> Torso_Side_Right; origin xyz=0 0 0 rpy=0.00 0.00 0.00 -> xyz=0 0 0 rpy=0.00 0.00 1.57

Commit message: new onshape with updated joint limits

File: kbot-v2-feet/robot.urdf (robot description, URDF)
Before this commit: robot kbotv2p0_nohands, 23 links, 22 joints
Links:
- link Torso_Side_Right: mass 13.322034 -> 13.516427
Joints:
- joint dof_left_ankle_02: limit lower=-0.785398 upper=0.296706 effort=17 velocity=12.566 -> lower=-1.256637 upper=0.226893 effort=17 velocity=12.566
- joint dof_right_ankle_02: limit lower=-0.296706 upper=0.785398 effort=17 velocity=12.566 -> lower=-0.226893 upper=1.256637 effort=17 velocity=12.566

File: kbot-v2/robot.urdf (robot description, URDF)
Before this commit: robot kbotv2p0_nohands, 23 links, 22 joints
Links:
- link Torso_Side_Right: mass 13.322034 -> 13.516427
Joints:
- joint dof_left_ankle_02: limit lower=-0.785398 upper=0.296706 effort=17 velocity=12.566 -> lower=-1.256637 upper=0.226893 effort=17 velocity=12.566
- joint dof_right_ankle_02: limit lower=-0.296706 upper=0.785398 effort=17 velocity=12.566 -> lower=-0.226893 upper=1.256637 effort=17 velocity=12.566

Commit message: update

File: kbot-v2-feet/robot.urdf (robot description, URDF)
Before this commit: robot kbotv2p0_nohands, 23 links, 22 joints
Joints:
- joint dof_left_ankle_02: limit lower=-1.256637 upper=0.226893 effort=17 velocity=12.566 -> lower=-1.256637 upper=0.226893 effort=17 velocity=37.699
- joint dof_left_elbow_02: limit lower=-2.478368 upper=0 effort=17 velocity=12.566 -> lower=-2.478368 upper=0 effort=17 velocity=37.699
- joint dof_left_hip_pitch_04: limit lower=-1.047198 upper=2.216568 effort=120 velocity=6.283 -> lower=-1.047198 upper=2.216568 effort=120 velocity=17.488
- joint dof_left_hip_roll_03: limit lower=-0.209440 upper=2.268928 effort=60 velocity=6.283 -> lower=-0.209440 upper=2.268928 effort=60 velocity=18.849
- joint dof_left_hip_yaw_03: limit lower=-1.570796 upper=1.570796 effort=60 velocity=6.283 -> lower=-1.570796 upper=1.570796 effort=60 velocity=18.849
- joint dof_left_knee_04: limit lower=0 upper=2.705260 effort=120 velocity=6.283 -> lower=0 upper=2.705260 effort=120 velocity=17.488
- joint dof_left_shoulder_pitch_03: limit lower=-1.047198 upper=3.490658 effort=60 velocity=6.283 -> lower=-1.047198 upper=3.490658 effort=60 velocity=18.849
- joint dof_left_shoulder_roll_03: limit lower=-0.383972 upper=1.658063 effort=60 velocity=6.283 -> lower=-0.383972 upper=1.658063 effort=60 velocity=18.849
- joint dof_left_shoulder_yaw_02: limit lower=-1.658063 upper=1.658063 effort=17 velocity=12.566 -> lower=-1.658063 upper=1.658063 effort=17 velocity=37.699
- joint dof_left_wrist_00: limit lower=-1.745329 upper=1.745329 effort=14 velocity=12.566 -> lower=-1.745329 upper=1.745329 effort=14 velocity=27.227
- joint dof_right_ankle_02: limit lower=-0.226893 upper=1.256637 effort=17 velocity=12.566 -> lower=-0.226893 upper=1.256637 effort=17 velocity=37.699
- joint dof_right_elbow_02: limit lower=0 upper=2.478368 effort=17 velocity=12.566 -> lower=0 upper=2.478368 effort=17 velocity=37.699
- joint dof_right_hip_pitch_04: limit lower=-2.216568 upper=1.047198 effort=120 velocity=6.283 -> lower=-2.216568 upper=1.047198 effort=120 velocity=17.488
- joint dof_right_hip_roll_03: limit lower=-2.268928 upper=0.209440 effort=60 velocity=6.283 -> lower=-2.268928 upper=0.209440 effort=60 velocity=18.849
- joint dof_right_hip_yaw_03: limit lower=-1.570796 upper=1.570796 effort=60 velocity=6.283 -> lower=-1.570796 upper=1.570796 effort=60 velocity=18.849
- joint dof_right_knee_04: limit lower=-2.705260 upper=0 effort=120 velocity=6.283 -> lower=-2.705260 upper=0 effort=120 velocity=17.488
- joint dof_right_shoulder_pitch_03: limit lower=-2.617994 upper=2.094395 effort=60 velocity=6.283 -> lower=-2.617994 upper=2.094395 effort=60 velocity=18.849
- joint dof_right_shoulder_roll_03: limit lower=-1.658063 upper=0.383972 effort=60 velocity=6.283 -> lower=-1.658063 upper=0.383972 effort=60 velocity=18.849
- joint dof_right_shoulder_yaw_02: limit lower=-1.658063 upper=1.658063 effort=17 velocity=12.566 -> lower=-1.658063 upper=1.658063 effort=17 velocity=37.699
- joint dof_right_wrist_00: limit lower=-1.745329 upper=1.745329 effort=14 velocity=12.566 -> lower=-1.745329 upper=1.745329 effort=14 velocity=27.227

File: kbot-v2/robot.urdf (robot description, URDF)
Before this commit: robot kbotv2p0_nohands, 23 links, 22 joints
Joints:
- joint dof_left_ankle_02: limit lower=-1.256637 upper=0.226893 effort=17 velocity=12.566 -> lower=-1.256637 upper=0.226893 effort=17 velocity=37.699
- joint dof_left_elbow_02: limit lower=-2.478368 upper=0 effort=17 velocity=12.566 -> lower=-2.478368 upper=0 effort=17 velocity=37.699
- joint dof_left_hip_pitch_04: limit lower=-1.047198 upper=2.216568 effort=120 velocity=6.283 -> lower=-1.047198 upper=2.216568 effort=120 velocity=17.488
- joint dof_left_hip_roll_03: limit lower=-0.209440 upper=2.268928 effort=60 velocity=6.283 -> lower=-0.209440 upper=2.268928 effort=60 velocity=18.849
- joint dof_left_hip_yaw_03: limit lower=-1.570796 upper=1.570796 effort=60 velocity=6.283 -> lower=-1.570796 upper=1.570796 effort=60 velocity=18.849
- joint dof_left_knee_04: limit lower=0 upper=2.705260 effort=120 velocity=6.283 -> lower=0 upper=2.705260 effort=120 velocity=17.488
- joint dof_left_shoulder_pitch_03: limit lower=-1.047198 upper=3.490658 effort=60 velocity=6.283 -> lower=-1.047198 upper=3.490658 effort=60 velocity=18.849
- joint dof_left_shoulder_roll_03: limit lower=-0.383972 upper=1.658063 effort=60 velocity=6.283 -> lower=-0.383972 upper=1.658063 effort=60 velocity=18.849
- joint dof_left_shoulder_yaw_02: limit lower=-1.658063 upper=1.658063 effort=17 velocity=12.566 -> lower=-1.658063 upper=1.658063 effort=17 velocity=37.699
- joint dof_left_wrist_00: limit lower=-1.745329 upper=1.745329 effort=14 velocity=12.566 -> lower=-1.745329 upper=1.745329 effort=14 velocity=27.227
- joint dof_right_ankle_02: limit lower=-0.226893 upper=1.256637 effort=17 velocity=12.566 -> lower=-0.226893 upper=1.256637 effort=17 velocity=37.699
- joint dof_right_elbow_02: limit lower=0 upper=2.478368 effort=17 velocity=12.566 -> lower=0 upper=2.478368 effort=17 velocity=37.699
- joint dof_right_hip_pitch_04: limit lower=-2.216568 upper=1.047198 effort=120 velocity=6.283 -> lower=-2.216568 upper=1.047198 effort=120 velocity=17.488
- joint dof_right_hip_roll_03: limit lower=-2.268928 upper=0.209440 effort=60 velocity=6.283 -> lower=-2.268928 upper=0.209440 effort=60 velocity=18.849
- joint dof_right_hip_yaw_03: limit lower=-1.570796 upper=1.570796 effort=60 velocity=6.283 -> lower=-1.570796 upper=1.570796 effort=60 velocity=18.849
- joint dof_right_knee_04: limit lower=-2.705260 upper=0 effort=120 velocity=6.283 -> lower=-2.705260 upper=0 effort=120 velocity=17.488
- joint dof_right_shoulder_pitch_03: limit lower=-2.617994 upper=2.094395 effort=60 velocity=6.283 -> lower=-2.617994 upper=2.094395 effort=60 velocity=18.849
- joint dof_right_shoulder_roll_03: limit lower=-1.658063 upper=0.383972 effort=60 velocity=6.283 -> lower=-1.658063 upper=0.383972 effort=60 velocity=18.849
- joint dof_right_shoulder_yaw_02: limit lower=-1.658063 upper=1.658063 effort=17 velocity=12.566 -> lower=-1.658063 upper=1.658063 effort=17 velocity=37.699
- joint dof_right_wrist_00: limit lower=-1.745329 upper=1.745329 effort=14 velocity=12.566 -> lower=-1.745329 upper=1.745329 effort=14 velocity=27.227
